File: hardware/v1-electronics/mcu_power_led.kicad_sch (KiCad schematic)
At the start: 32 parts, among them IC1 IS31FL3741A-QFLS4-TR, J1 Conn_01x01_Pin, J2 Conn_01x01_Socket

Commit message: feat(v1 hardware): Add new LED Matrix driver
- added the symbol for 3733
- added circuit for 3733
- have not removed: old matrix and 3741A symbol & circuits
Parts:
- removed IC1: IS31FL3741A-QFLS4-TR, QFN40P700X700X80-61N-D, symbol Lumissil Microsystems IS31FL3741A-QFLS4-TR:IS31FL3741A-QFLS4-TR
- removed J1: Conn_01x01_Pin, symbol Connector:Conn_01x01_Pin
- removed J2: Conn_01x01_Socket, symbol Connector:Conn_01x01_Socket
- added IC2: IS31FL3741A-QFLS4-TR, QFN40P700X700X80-61N-D, symbol Lumissil Microsystems:IS31FL3741A-QFLS4-TR
Connections:
- net GND: now also IC2.12 (GND_1), IC2.36 (GND_2), IC2.55 (GND_3), IC2.8 (ADDR)
- net I2C1_SCL: now also IC2.10 (SCL)
- net I2C1_SDA: now also IC2.9 (SDA)
- net IS31FL3741A_INTB: now also IC2.7 (INTB)
- net IS31FL3741A_SDB: now also IC2.11 (SDB)
- net V_SYS: now also IC2.14 (AVCC), IC2.15 (PVCC_1), IC2.25 (PVCC_2)
- net at R67.2: now also IC2.13 (ISET)
