File: hardware/v1-electronics/led_matrix.kicad_sch (KiCad schematic)
At the start: 47 parts, among them IC1 IS31FL3741A-QFLS4-TR

Commit message: feat(v1 hardware): LED Matrix refactor start
- refactored RGBW LED schematic symbol.
- realize that IS31FL3741A will need to be replaced.
Parts:
- removed C27, C28, C29, C30, C31, C32, C34: C_Small, symbol Device:C_Small
- removed IC1: IS31FL3741A-QFLS4-TR, QFN40P700X700X80-61N-D, symbol Lumissil Microsystems IS31FL3741A-QFLS4-TR:IS31FL3741A-QFLS4-TR
- removed R33, R41, R42: R_Small, symbol Device:R_Small
- added LED14, LED21, LED28, LED35, LED42, LED43, LED44, LED45, LED46, LED47, LED48, LED49, LED50, LED51, LED52, LED53, LED54, LED55, LED56, LED57, LED58, LED59, LED60, LED61, LED62, LED63, LED64, LED65, LED66, LED67, LED68, LED69, LED7, LED70, LED71, LED72, LED73, LED74, LED75, LED76, LED77, LED78, LED79, LED80, LED81, LED82, LED83, LED84, LED85, LED86, LED87, LED88, LED89, LED90: LTST-FC12WEGBD-5A, LTSTFC12WEGBD5A, symbol Lite-On LTST-FC12WEGBD-5A:LTST-FC12WEGBD-5A
- added R100, R101, R104, R105, R106, R107, R108, R109, R110, R111, R112, R43, R44, R45, R46, R47, R48, R49, R50, R51, R52, R53, R54, R55, R56, R57, R58, R59, R60, R61, R62, R63, R64, R65, R66, R68, R69, R70, R71, R72, R73, R74, R75, R76, R77, R78, R79, R80, R81, R82, R83, R84, R85, R86, R87, R88, R89, R90, R91, R92, R93, R94, R95, R96, R97, R98, R99: R_Small, symbol Device:R_Small
- renumbered LED15 to LED10, LED16 to LED11, LED27 to LED12, LED28 to LED13, LED3 to LED15, LED9 to LED16, LED29 to LED19, LED7 to LED2, LED30 to LED20, LED4 to LED22, LED10 to LED23, LED19 to LED24, LED20 to LED25, LED31 to LED26, LED32 to LED27, LED5 to LED29, LED13 to LED3, LED11 to LED30, LED21 to LED31, LED22 to LED32, LED6 to LED36, LED12 to LED37, LED23 to LED38, LED24 to LED39, LED14 to LED4, LED35 to LED40, LED36 to LED41, LED25 to LED5, LED26 to LED6, LED2 to LED8, LED8 to LED9
Connections:
- net at LED39.1 (BLUE): now also LED11.1 (BLUE), LED18.1 (BLUE), LED25.1 (BLUE), LED32.1 (BLUE), LED4.1 (BLUE), R55.2
- net at LED39.2 (GREEN): now also LED11.2 (GREEN), LED18.2 (GREEN), LED25.2 (GREEN), LED32.2 (GREEN), LED4.2 (GREEN), R56.1
- net at LED39.3 (RED): now also LED11.3 (RED), LED18.3 (RED), LED25.3 (RED), LED32.3 (RED), LED4.3 (RED), R57.1
- net at LED39.4 (WHITE): now also LED11.4 (WHITE), LED18.4 (WHITE), LED25.4 (WHITE), LED32.4 (WHITE), LED4.4 (WHITE), R58.1
- net SW6: now reaches LED39.5 (ANODE)
- net SW6: now also LED36.5 (ANODE), LED37.5 (ANODE), LED38.5 (ANODE), LED40.5 (ANODE), LED41.5 (ANODE), LED42.5 (ANODE), LED74.5 (ANODE), LED75.5 (ANODE), LED87.5 (ANODE)
- net at LED9.1 (BLUE): now also LED16.1 (BLUE), LED2.1 (BLUE), LED23.1 (BLUE), LED30.1 (BLUE), LED37.1 (BLUE), R47.2
- net at LED9.2 (GREEN): now also LED16.2 (GREEN), LED2.2 (GREEN), LED23.2 (GREEN), LED30.2 (GREEN), LED37.2 (GREEN), R48.1
- net at LED9.3 (RED): now also LED16.3 (RED), LED2.3 (RED), LED23.3 (RED), LED30.3 (RED), LED37.3 (RED), R49.1
- net at LED9.4 (WHITE): now also LED16.4 (WHITE), LED2.4 (WHITE), LED23.4 (WHITE), LED30.4 (WHITE), LED37.4 (WHITE), R50.1
- net SW2: now reaches LED9.5 (ANODE)
- net SW2: now also LED10.5 (ANODE), LED11.5 (ANODE), LED12.5 (ANODE), LED13.5 (ANODE), LED8.5 (ANODE), LED14.5 (ANODE), LED66.5 (ANODE), LED67.5 (ANODE), LED83.5 (ANODE)
- net at LED36.1 (BLUE): now also LED1.1 (BLUE), LED15.1 (BLUE), LED22.1 (BLUE), LED29.1 (BLUE), LED8.1 (BLUE), R43.2
- net at LED36.2 (GREEN): now also LED1.2 (GREEN), LED15.2 (GREEN), LED22.2 (GREEN), LED29.2 (GREEN), LED8.2 (GREEN), R44.1
- net at LED36.3 (RED): now also LED1.3 (RED), LED15.3 (RED), LED22.3 (RED), LED29.3 (RED), LED8.3 (RED), R45.1
- net at LED36.4 (WHITE): now also LED1.4 (WHITE), LED15.4 (WHITE), LED22.4 (WHITE), LED29.4 (WHITE), LED8.4 (WHITE), R46.1
- net SW5: now reaches LED30.5 (ANODE)
- net SW5: now also LED29.5 (ANODE), LED31.5 (ANODE), LED32.5 (ANODE), LED33.5 (ANODE), LED34.5 (ANODE), LED35.5 (ANODE), LED72.5 (ANODE), LED73.5 (ANODE), LED86.5 (ANODE)
- net at LED27.1 (BLUE): now also LED13.1 (BLUE), LED20.1 (BLUE), LED34.1 (BLUE), LED41.1 (BLUE), LED6.1 (BLUE), R63.2
- net at LED27.2 (GREEN): now also LED13.2 (GREEN), LED20.2 (GREEN), LED34.2 (GREEN), LED41.2 (GREEN), LED6.2 (GREEN), R64.1
- net at LED27.3 (RED): now also LED13.3 (RED), LED20.3 (RED), LED34.3 (RED), LED41.3 (RED), LED6.3 (RED), R65.1
- net at LED27.4 (WHITE): now also LED13.4 (WHITE), LED20.4 (WHITE), LED34.4 (WHITE), LED41.4 (WHITE), LED6.4 (WHITE), R66.1
- net SW4: now reaches LED27.5 (ANODE)
- net SW4: now also LED22.5 (ANODE), LED23.5 (ANODE), LED24.5 (ANODE), LED25.5 (ANODE), LED26.5 (ANODE), LED28.5 (ANODE), LED70.5 (ANODE), LED71.5 (ANODE), LED85.5 (ANODE)
- net at LED5.1 (BLUE): now also LED12.1 (BLUE), LED19.1 (BLUE), LED26.1 (BLUE), LED33.1 (BLUE), LED40.1 (BLUE), R59.2
- net at LED5.2 (GREEN): now also LED12.2 (GREEN), LED19.2 (GREEN), LED26.2 (GREEN), LED33.2 (GREEN), LED40.2 (GREEN), R60.1
- net at LED5.3 (RED): now also LED12.3 (RED), LED19.3 (RED), LED26.3 (RED), LED33.3 (RED), LED40.3 (RED), R61.1
- net at LED5.4 (WHITE): now also LED12.4 (WHITE), LED19.4 (WHITE), LED26.4 (WHITE), LED33.4 (WHITE), LED40.4 (WHITE), R62.1
- net SW1: now reaches LED5.5 (ANODE)
- net SW1: now also LED1.5 (ANODE), LED2.5 (ANODE), LED3.5 (ANODE), LED4.5 (ANODE), LED6.5 (ANODE), LED64.5 (ANODE), LED65.5 (ANODE), LED7.5 (ANODE), LED82.5 (ANODE)
- net SW3: now reaches LED20.5 (ANODE)
- net SW3: now also LED15.5 (ANODE), LED16.5 (ANODE), LED17.5 (ANODE), LED18.5 (ANODE), LED19.5 (ANODE), LED21.5 (ANODE), LED68.5 (ANODE), LED69.5 (ANODE), LED84.5 (ANODE)
- net at LED17.1 (BLUE): now also LED10.1 (BLUE), LED24.1 (BLUE), LED3.1 (BLUE), LED31.1 (BLUE), LED38.1 (BLUE), R51.2
- net at LED17.2 (GREEN): now also LED10.2 (GREEN), LED24.2 (GREEN), LED3.2 (GREEN), LED31.2 (GREEN), LED38.2 (GREEN), R52.1
- net at LED17.3 (RED): now also LED10.3 (RED), LED24.3 (RED), LED3.3 (RED), LED31.3 (RED), LED38.3 (RED), R53.1
- net at LED17.4 (WHITE): now also LED10.4 (WHITE), LED24.4 (WHITE), LED3.4 (WHITE), LED31.4 (WHITE), LED38.4 (WHITE), R54.1
- new net: LED64.1 (BLUE), LED66.1 (BLUE), LED68.1 (BLUE), LED70.1 (BLUE), LED72.1 (BLUE), LED74.1 (BLUE), LED76.1 (BLUE), LED78.1 (BLUE), LED80.1 (BLUE), R104.2
- new net: LED64.2 (GREEN), LED66.2 (GREEN), LED68.2 (GREEN), LED70.2 (GREEN), LED72.2 (GREEN), LED74.2 (GREEN), LED76.2 (GREEN), LED78.2 (GREEN), LED80.2 (GREEN), R105.1
- new net: LED64.3 (RED), LED66.3 (RED), LED68.3 (RED), LED70.3 (RED), LED72.3 (RED), LED74.3 (RED), LED76.3 (RED), LED78.3 (RED), LED80.3 (RED), R106.1
- new net: LED64.4 (WHITE), LED66.4 (WHITE), LED68.4 (WHITE), LED70.4 (WHITE), LED72.4 (WHITE), LED74.4 (WHITE), LED76.4 (WHITE), LED78.4 (WHITE), LED80.4 (WHITE), R107.1
- new net: LED45.1 (BLUE), LED52.1 (BLUE), LED59.1 (BLUE), R82.2
- new net: LED45.2 (GREEN), LED52.2 (GREEN), LED59.2 (GREEN), R83.1
- new net: LED45.3 (RED), LED52.3 (RED), LED59.3 (RED), R84.1
- new net: LED45.4 (WHITE), LED52.4 (WHITE), LED59.4 (WHITE), R85.1
- new net: LED46.1 (BLUE), LED53.1 (BLUE), LED60.1 (BLUE), R86.2
- new net: LED46.2 (GREEN), LED53.2 (GREEN), LED60.2 (GREEN), R87.1
- new net: LED46.3 (RED), LED53.3 (RED), LED60.3 (RED), R88.1
- new net: LED46.4 (WHITE), LED53.4 (WHITE), LED60.4 (WHITE), R89.1
- new net: LED65.3 (RED), LED67.3 (RED), LED69.3 (RED), LED71.3 (RED), LED73.3 (RED), LED75.3 (RED), LED77.3 (RED), LED79.3 (RED), LED81.3 (RED), R110.1
- new net: LED82.2 (GREEN), LED83.2 (GREEN), LED84.2 (GREEN), LED85.2 (GREEN), LED86.2 (GREEN), LED87.2 (GREEN), LED88.2 (GREEN), LED89.2 (GREEN), LED90.2 (GREEN), R73.1
- new net: LED43.1 (BLUE), LED50.1 (BLUE), LED57.1 (BLUE), R74.2
- new net: LED43.2 (GREEN), LED50.2 (GREEN), LED57.2 (GREEN), R75.1
- new net: LED43.3 (RED), LED50.3 (RED), LED57.3 (RED), R76.1
- new net: LED43.4 (WHITE), LED50.4 (WHITE), LED57.4 (WHITE), R77.1
- new net: LED48.1 (BLUE), LED55.1 (BLUE), LED62.1 (BLUE), R94.2
- new net: LED48.2 (GREEN), LED55.2 (GREEN), LED62.2 (GREEN), R95.1
- new net: LED48.3 (RED), LED55.3 (RED), LED62.3 (RED), R96.1
- new net: LED48.4 (WHITE), LED55.4 (WHITE), LED62.4 (WHITE), R97.1
- new net: LED65.1 (BLUE), LED67.1 (BLUE), LED69.1 (BLUE), LED71.1 (BLUE), LED73.1 (BLUE), LED75.1 (BLUE), LED77.1 (BLUE), LED79.1 (BLUE), LED81.1 (BLUE), R108.2
- new net: LED65.2 (GREEN), LED67.2 (GREEN), LED69.2 (GREEN), LED71.2 (GREEN), LED73.2 (GREEN), LED75.2 (GREEN), LED77.2 (GREEN), LED79.2 (GREEN), LED81.2 (GREEN), R109.1
- new net: LED65.4 (WHITE), LED67.4 (WHITE), LED69.4 (WHITE), LED71.4 (WHITE), LED73.4 (WHITE), LED75.4 (WHITE), LED77.4 (WHITE), LED79.4 (WHITE), LED81.4 (WHITE), R111.1
- new net: LED14.4 (WHITE), LED21.4 (WHITE), LED28.4 (WHITE), LED35.4 (WHITE), LED42.4 (WHITE), LED7.4 (WHITE), R71.1
- new net: LED14.1 (BLUE), LED21.1 (BLUE), LED28.1 (BLUE), LED35.1 (BLUE), LED42.1 (BLUE), LED7.1 (BLUE), R68.2
- new net: LED14.2 (GREEN), LED21.2 (GREEN), LED28.2 (GREEN), LED35.2 (GREEN), LED42.2 (GREEN), LED7.2 (GREEN), R69.1
- new net: LED14.3 (RED), LED21.3 (RED), LED28.3 (RED), LED35.3 (RED), LED42.3 (RED), LED7.3 (RED), R70.1
- new net: LED82.3 (RED), LED83.3 (RED), LED84.3 (RED), LED85.3 (RED), LED86.3 (RED), LED87.3 (RED), LED88.3 (RED), LED89.3 (RED), LED90.3 (RED), R112.1
- new net: LED82.1 (BLUE), LED83.1 (BLUE), LED84.1 (BLUE), LED85.1 (BLUE), LED86.1 (BLUE), LED87.1 (BLUE), LED88.1 (BLUE), LED89.1 (BLUE), LED90.1 (BLUE), R72.2
- new net: LED49.3 (RED), LED56.3 (RED), LED63.3 (RED), R100.1
- new net: LED47.4 (WHITE), LED54.4 (WHITE), LED61.4 (WHITE), R93.1
- new net: LED44.1 (BLUE), LED51.1 (BLUE), LED58.1 (BLUE), R78.2
- new net: LED44.2 (GREEN), LED51.2 (GREEN), LED58.2 (GREEN), R79.1
- new net: LED44.3 (RED), LED51.3 (RED), LED58.3 (RED), R80.1
- new net: LED44.4 (WHITE), LED51.4 (WHITE), LED58.4 (WHITE), R81.1
- new net: LED47.3 (RED), LED54.3 (RED), LED61.3 (RED), R92.1
- new net: LED47.1 (BLUE), LED54.1 (BLUE), LED61.1 (BLUE), R90.2
- new net: LED47.2 (GREEN), LED54.2 (GREEN), LED61.2 (GREEN), R91.1
- new net: LED49.1 (BLUE), LED56.1 (BLUE), LED63.1 (BLUE), R98.2
- new net: LED49.2 (GREEN), LED56.2 (GREEN), LED63.2 (GREEN), R99.1
- new net: LED49.4 (WHITE), LED56.4 (WHITE), LED63.4 (WHITE), R101.1
- new net CS10_G: R52.2, R83.2
- new net CS11_R: R53.2, R84.2
- new net CS12_W: R54.2, R85.2
- new net CS13_B: R55.1, R86.1
- new net CS14_G: R56.2, R87.2
- new net CS15_R: R57.2, R88.2
- new net CS16_W: R58.2, R89.2
- new net CS17_B: R59.1, R90.1
- new net CS18_G: R60.2, R91.2
- new net CS19_R: R61.2, R92.2
- new net CS1_B: R43.1, R74.1
- new net CS20_W: R62.2, R93.2
- new net CS21_B: R63.1, R94.1
- new net CS22_G: R64.2, R95.2
- new net CS23_R: R65.2, R96.2
- new net CS24_W: R66.2, R97.2
- new net CS25_B: R68.1, R98.1
- new net CS26_G: R69.2, R99.2
- new net CS27_R: R100.2, R70.2
- new net CS28_W: R101.2, R71.2
- new net CS29_B: R72.1
- new net CS2_G: R44.2, R75.2
- new net CS30_G: R73.2
- new net CS31_B: R104.1
- new net CS32_G: R105.2
- new net CS33_R: R106.2
- new net CS34_W: R107.2
- new net CS35_B: R108.1
- new net CS36_G: R109.2
- new net CS37_R: R110.2
- new net CS38_W: R111.2
- new net CS39_R: R112.2
- new net CS3_R: R45.2, R76.2
- new net CS4_W: R46.2, R77.2
- new net CS5_B: R47.1, R78.1
- new net CS6_G: R48.2, R79.2
- new net CS7_R: R49.2, R80.2
- new net CS8_W: R50.2, R81.2
- new net CS9_B: R51.1, R82.1
- new net SW7: LED43.5 (ANODE), LED44.5 (ANODE), LED45.5 (ANODE), LED46.5 (ANODE), LED47.5 (ANODE), LED48.5 (ANODE), LED49.5 (ANODE), LED76.5 (ANODE), LED77.5 (ANODE), LED88.5 (ANODE)
- new net SW8: LED50.5 (ANODE), LED51.5 (ANODE), LED52.5 (ANODE), LED53.5 (ANODE), LED54.5 (ANODE), LED55.5 (ANODE), LED56.5 (ANODE), LED78.5 (ANODE), LED79.5 (ANODE), LED89.5 (ANODE)
- new net SW9: LED57.5 (ANODE), LED58.5 (ANODE), LED59.5 (ANODE), LED60.5 (ANODE), LED61.5 (ANODE), LED62.5 (ANODE), LED63.5 (ANODE), LED80.5 (ANODE), LED81.5 (ANODE), LED90.5 (ANODE)
Other:
- note added: "Because our matrix is divisible by 4, and our matrix address led's interestingly we're haing some layout problems"
- note added: "In the next verision I can do we'll cascade IS31FL3733 and IS31FL3737 drivers"
- note added: "Page 0"
- note added: "Page 0 + 1 Incomplete Rows"
- note added: "Page 1 Bank 1"
- note added: "Page 1 Bank 2"
- note added: "The matrix I've layed out thus far is too small.Should be double the size."
- note removed: "Some thought needs to be done as to what V_IO/MCU should be"

Commit message: feat(v1 hardware): RGBW LED matrix halve 1
Parts:
- removed LED43, LED44, LED45, LED46, LED47, LED48, LED49, LED50, LED51, LED52, LED53, LED54, LED55, LED56, LED57, LED58, LED59, LED60, LED61, LED62, LED63, LED64, LED65, LED66, LED67, LED68, LED69, LED70, LED71, LED72, LED73, LED74, LED75, LED76, LED77, LED78, LED79, LED80, LED81, LED82, LED83, LED84, LED85, LED86, LED87, LED88, LED89, LED90: LTST-FC12WEGBD-5A, LTSTFC12WEGBD5A, symbol Lite-On LTST-FC12WEGBD-5A:LTST-FC12WEGBD-5A
- removed R100, R101, R104, R105, R106, R107, R108, R109, R110, R111, R112, R43, R44, R45, R46, R47, R48, R49, R50, R51, R52, R53, R54, R55, R56, R57, R58, R59, R60, R61, R62, R63, R64, R65, R66, R68, R70, R71, R72, R73, R74, R75, R76, R77, R78, R79, R80, R81, R82, R83, R84, R85, R86, R87, R88, R89, R90, R91, R92, R93, R94, R95, R96, R97, R98, R99: R_Small, symbol Device:R_Small
- added R119, R120, R121, R122, R123, R124, R125, R126, R127, R128, R129, R130, R131, R132, R133, R134, R135, R136, R137, R138, R139, R140, R141, R142, R143, R144, R145, R146, R147, R177, R67: R_Small, symbol Device:R_Small
Connections:
- net CS26_G: no longer names the net of R69.2
- net CS26_G: now also LED1.1 (BLUE), LED13.1 (BLUE), LED17.1 (BLUE), LED21.1 (BLUE), LED25.1 (BLUE), LED29.1 (BLUE), LED33.1 (BLUE), LED37.1 (BLUE), LED41.1 (BLUE), LED5.1 (BLUE), LED9.1 (BLUE)
- net SW1 renamed SW1_1
- net SW1_1: no longer LED5.5 (ANODE), LED6.5 (ANODE), LED7.5 (ANODE)
- net SW2 renamed SW3_1
- net SW3_1: no longer LED13.5 (ANODE), LED14.5 (ANODE), LED8.5 (ANODE)
- net SW3 renamed SW5_1
- net SW5_1: no longer LED15.5 (ANODE), LED16.5 (ANODE), LED21.5 (ANODE)
- net SW4 renamed SW7_1
- net SW7_1: no longer LED22.5 (ANODE), LED23.5 (ANODE), LED24.5 (ANODE)
- net SW5 renamed SW8_1
- net SW8_1: no longer LED33.5 (ANODE), LED34.5 (ANODE), LED35.5 (ANODE)
- net SW6 renamed SW10_1
- net SW10_1: no longer LED36.5 (ANODE), LED41.5 (ANODE), LED42.5 (ANODE)
- new net: LED11.1 (BLUE), LED15.1 (BLUE), LED19.1 (BLUE), LED23.1 (BLUE), LED27.1 (BLUE), LED3.1 (BLUE), LED31.1 (BLUE), LED35.1 (BLUE), LED39.1 (BLUE), LED7.1 (BLUE), R124.2
- new net: LED11.2 (GREEN), LED15.2 (GREEN), LED19.2 (GREEN), LED23.2 (GREEN), LED27.2 (GREEN), LED3.2 (GREEN), LED31.2 (GREEN), LED35.2 (GREEN), LED39.2 (GREEN), LED7.2 (GREEN), R125.2
- new net: LED11.3 (RED), LED15.3 (RED), LED19.3 (RED), LED23.3 (RED), LED27.3 (RED), LED3.3 (RED), LED31.3 (RED), LED35.3 (RED), LED39.3 (RED), LED7.3 (RED), R126.2
- new net: LED11.4 (WHITE), LED15.4 (WHITE), LED19.4 (WHITE), LED23.4 (WHITE), LED27.4 (WHITE), LED3.4 (WHITE), LED31.4 (WHITE), LED35.4 (WHITE), LED39.4 (WHITE), LED7.4 (WHITE), R127.2
- new net: LED10.1 (BLUE), LED14.1 (BLUE), LED18.1 (BLUE), LED2.1 (BLUE), LED22.1 (BLUE), LED26.1 (BLUE), LED30.1 (BLUE), LED34.1 (BLUE), LED38.1 (BLUE), LED42.1 (BLUE), LED6.1 (BLUE), R120.2
- new net: LED10.2 (GREEN), LED14.2 (GREEN), LED18.2 (GREEN), LED2.2 (GREEN), LED22.2 (GREEN), LED26.2 (GREEN), LED30.2 (GREEN), LED34.2 (GREEN), LED38.2 (GREEN), LED42.2 (GREEN), LED6.2 (GREEN), R121.2
- new net: LED10.3 (RED), LED14.3 (RED), LED18.3 (RED), LED2.3 (RED), LED22.3 (RED), LED26.3 (RED), LED30.3 (RED), LED34.3 (RED), LED38.3 (RED), LED42.3 (RED), LED6.3 (RED), R122.2
- new net: LED10.4 (WHITE), LED14.4 (WHITE), LED18.4 (WHITE), LED2.4 (WHITE), LED22.4 (WHITE), LED26.4 (WHITE), LED30.4 (WHITE), LED34.4 (WHITE), LED38.4 (WHITE), LED42.4 (WHITE), LED6.4 (WHITE), R123.2
- new net: LED1.2 (GREEN), LED13.2 (GREEN), LED17.2 (GREEN), LED21.2 (GREEN), LED25.2 (GREEN), LED29.2 (GREEN), LED33.2 (GREEN), LED37.2 (GREEN), LED41.2 (GREEN), LED5.2 (GREEN), LED9.2 (GREEN), R177.2
- new net: LED1.3 (RED), LED13.3 (RED), LED17.3 (RED), LED21.3 (RED), LED25.3 (RED), LED29.3 (RED), LED33.3 (RED), LED37.3 (RED), LED41.3 (RED), LED5.3 (RED), LED9.3 (RED), R67.2
- new net: LED1.4 (WHITE), LED13.4 (WHITE), LED17.4 (WHITE), LED21.4 (WHITE), LED25.4 (WHITE), LED29.4 (WHITE), LED33.4 (WHITE), LED37.4 (WHITE), LED41.4 (WHITE), LED5.4 (WHITE), LED9.4 (WHITE), R119.2
- new net: LED12.4 (WHITE), LED16.4 (WHITE), LED20.4 (WHITE), LED24.4 (WHITE), LED28.4 (WHITE), LED32.4 (WHITE), LED36.4 (WHITE), LED4.4 (WHITE), LED40.4 (WHITE), LED8.4 (WHITE), R131.2
- new net: LED12.1 (BLUE), LED16.1 (BLUE), LED20.1 (BLUE), LED24.1 (BLUE), LED28.1 (BLUE), LED32.1 (BLUE), LED36.1 (BLUE), LED4.1 (BLUE), LED40.1 (BLUE), LED8.1 (BLUE), R128.2
- new net: LED12.2 (GREEN), LED16.2 (GREEN), LED20.2 (GREEN), LED24.2 (GREEN), LED28.2 (GREEN), LED32.2 (GREEN), LED36.2 (GREEN), LED4.2 (GREEN), LED40.2 (GREEN), LED8.2 (GREEN), R129.2
- new net: LED12.3 (RED), LED16.3 (RED), LED20.3 (RED), LED24.3 (RED), LED28.3 (RED), LED32.3 (RED), LED36.3 (RED), LED4.3 (RED), LED40.3 (RED), LED8.3 (RED), R130.2
- new net CS10_G_1: R125.1
- new net CS10_G_2: R141.1
- new net CS11_R_1: R126.1
- new net CS11_R_2: R142.1
- new net CS12_W_1: R127.1
- new net CS12_W_2: R143.1
- new net CS13_B_1: R128.1
- new net CS13_B_2: R144.1
- new net CS14_G_1: R129.1
- new net CS14_G_2: R145.1
- new net CS15_R_1: R130.1
- new net CS15_R_2: R146.1
- new net CS16_W_1: R131.1
- new net CS16_W_2: R147.1
- new net CS1_B_1: R69.1
- new net CS1_B_2: R132.1
- new net CS2_G_1: R177.1
- new net CS2_G_2: R133.1
- new net CS3_R_1: R67.1
- new net CS3_R_2: R134.1
- new net CS4_W_1: R119.1
- new net CS4_W_2: R135.1
- new net CS5_B_1: R120.1
- new net CS5_B_2: R136.1
- new net CS6_G_1: R121.1
- new net CS6_G_2: R137.1
- new net CS7_R_1: R122.1
- new net CS7_R_2: R138.1
- new net CS8_W_1: R123.1
- new net CS8_W_2: R139.1
- new net CS9_B_1: R124.1
- new net CS9_B_2: R140.1
- new net SW11_1: LED41.5 (ANODE), LED42.5 (ANODE)
- new net SW2_1: LED5.5 (ANODE), LED6.5 (ANODE), LED7.5 (ANODE), LED8.5 (ANODE)
- new net SW4_1: LED13.5 (ANODE), LED14.5 (ANODE), LED15.5 (ANODE), LED16.5 (ANODE)
- new net SW6_1: LED21.5 (ANODE), LED22.5 (ANODE), LED23.5 (ANODE), LED24.5 (ANODE)
- new net SW9_1: LED33.5 (ANODE), LED34.5 (ANODE), LED35.5 (ANODE), LED36.5 (ANODE)
Other:
- note added: "RGBW LED Matrix Halve 1"
- note added: "RGBW LED Matrix Halve 2"
- note removed: "Because our matrix is divisible by 4, and our matrix address led's interestingly we're haing some layout problems"
- note removed: "Page 0"
- note removed: "Page 0 + 1 Incomplete Rows"
- note removed: "Page 1 Bank 1"
- note removed: "Page 1 Bank 2"

Commit message: feat(v1 hardware):second half of LED Matrix
Parts:
- added LED43, LED44, LED45, LED46, LED47, LED48, LED49, LED50, LED51, LED52, LED53, LED54, LED55, LED56, LED57, LED58, LED59, LED60, LED61, LED62, LED63, LED64, LED65, LED66, LED67, LED68, LED69, LED70, LED71, LED72, LED73, LED74, LED75, LED76, LED77, LED78, LED79, LED80, LED81, LED82, LED83, LED84: LTST-FC12WEGBD-5A, LTSTFC12WEGBD5A, symbol Lite-On LTST-FC12WEGBD-5A:LTST-FC12WEGBD-5A
- renumbered LED1 to LED1_1, LED2 to LED2_1, LED3 to LED3_1
Connections:
- net SW10_2: now also LED79.5 (ANODE), LED80.5 (ANODE), LED81.5 (ANODE), LED82.5 (ANODE)
- net SW11_2: now also LED83.5 (ANODE), LED84.5 (ANODE)
- net SW1_2: now also LED43.5 (ANODE), LED44.5 (ANODE), LED45.5 (ANODE), LED46.5 (ANODE)
- net SW2_2: now also LED47.5 (ANODE), LED48.5 (ANODE), LED49.5 (ANODE), LED50.5 (ANODE)
- net SW3_2: now also LED51.5 (ANODE), LED52.5 (ANODE), LED53.5 (ANODE), LED54.5 (ANODE)
- net SW4_2: now also LED55.5 (ANODE), LED56.5 (ANODE), LED57.5 (ANODE), LED58.5 (ANODE)
- net SW5_2: now also LED59.5 (ANODE), LED60.5 (ANODE), LED61.5 (ANODE), LED62.5 (ANODE)
- net SW6_2: now also LED63.5 (ANODE), LED64.5 (ANODE), LED65.5 (ANODE), LED66.5 (ANODE)
- net SW7_2: now also LED67.5 (ANODE), LED68.5 (ANODE), LED69.5 (ANODE), LED70.5 (ANODE)
- net SW8_2: now also LED71.5 (ANODE), LED72.5 (ANODE), LED73.5 (ANODE), LED74.5 (ANODE)
- net SW9_2: now also LED75.5 (ANODE), LED76.5 (ANODE), LED77.5 (ANODE), LED78.5 (ANODE)
- net at R147.2: now also LED46.4 (WHITE), LED50.4 (WHITE), LED54.4 (WHITE), LED58.4 (WHITE), LED62.4 (WHITE), LED66.4 (WHITE), LED70.4 (WHITE), LED74.4 (WHITE), LED78.4 (WHITE), LED82.4 (WHITE)
- net at R146.2: now also LED46.3 (RED), LED50.3 (RED), LED54.3 (RED), LED58.3 (RED), LED62.3 (RED), LED66.3 (RED), LED70.3 (RED), LED74.3 (RED), LED78.3 (RED), LED82.3 (RED)
- net at R137.2: now also LED44.2 (GREEN), LED48.2 (GREEN), LED52.2 (GREEN), LED56.2 (GREEN), LED60.2 (GREEN), LED64.2 (GREEN), LED68.2 (GREEN), LED72.2 (GREEN), LED76.2 (GREEN), LED80.2 (GREEN), LED84.2 (GREEN)
- net at R138.2: now also LED44.3 (RED), LED48.3 (RED), LED52.3 (RED), LED56.3 (RED), LED60.3 (RED), LED64.3 (RED), LED68.3 (RED), LED72.3 (RED), LED76.3 (RED), LED80.3 (RED), LED84.3 (RED)
- net at R134.2: now also LED43.3 (RED), LED47.3 (RED), LED51.3 (RED), LED55.3 (RED), LED63.3 (RED), LED67.3 (RED), LED71.3 (RED), LED75.3 (RED), LED79.3 (RED), LED83.3 (RED)
- net at R136.2: now also LED44.1 (BLUE), LED48.1 (BLUE), LED52.1 (BLUE), LED56.1 (BLUE), LED60.1 (BLUE), LED64.1 (BLUE), LED68.1 (BLUE), LED72.1 (BLUE), LED76.1 (BLUE), LED80.1 (BLUE), LED84.1 (BLUE)
- net at R139.2: now also LED44.4 (WHITE), LED48.4 (WHITE), LED52.4 (WHITE), LED56.4 (WHITE), LED60.4 (WHITE), LED64.4 (WHITE), LED68.4 (WHITE), LED72.4 (WHITE), LED76.4 (WHITE), LED80.4 (WHITE), LED84.4 (WHITE)
- net at R143.2: now also LED45.4 (WHITE), LED49.4 (WHITE), LED53.4 (WHITE), LED57.4 (WHITE), LED61.4 (WHITE), LED65.4 (WHITE), LED69.4 (WHITE), LED73.4 (WHITE), LED77.4 (WHITE), LED81.4 (WHITE)
- net at R144.2: now also LED46.1 (BLUE), LED50.1 (BLUE), LED54.1 (BLUE), LED58.1 (BLUE), LED62.1 (BLUE), LED66.1 (BLUE), LED70.1 (BLUE), LED74.1 (BLUE), LED78.1 (BLUE), LED82.1 (BLUE)
- net at R145.2: now also LED46.2 (GREEN), LED50.2 (GREEN), LED54.2 (GREEN), LED58.2 (GREEN), LED62.2 (GREEN), LED66.2 (GREEN), LED70.2 (GREEN), LED74.2 (GREEN), LED78.2 (GREEN), LED82.2 (GREEN)
- net at R133.2: now also LED43.2 (GREEN), LED47.2 (GREEN), LED51.2 (GREEN), LED55.2 (GREEN), LED63.2 (GREEN), LED67.2 (GREEN), LED71.2 (GREEN), LED75.2 (GREEN), LED79.2 (GREEN), LED83.2 (GREEN)
- net at R140.2: now also LED45.1 (BLUE), LED49.1 (BLUE), LED53.1 (BLUE), LED57.1 (BLUE), LED61.1 (BLUE), LED65.1 (BLUE), LED69.1 (BLUE), LED73.1 (BLUE), LED77.1 (BLUE), LED81.1 (BLUE)
- net at R132.2: now also LED43.1 (BLUE), LED47.1 (BLUE), LED51.1 (BLUE), LED55.1 (BLUE), LED63.1 (BLUE), LED67.1 (BLUE), LED71.1 (BLUE), LED75.1 (BLUE), LED79.1 (BLUE), LED83.1 (BLUE)
- net at R142.2: now also LED45.3 (RED), LED49.3 (RED), LED53.3 (RED), LED57.3 (RED), LED61.3 (RED), LED65.3 (RED), LED69.3 (RED), LED73.3 (RED), LED77.3 (RED), LED81.3 (RED)
- net at R135.2: now also LED43.4 (WHITE), LED47.4 (WHITE), LED51.4 (WHITE), LED55.4 (WHITE), LED63.4 (WHITE), LED67.4 (WHITE), LED71.4 (WHITE), LED75.4 (WHITE), LED79.4 (WHITE), LED83.4 (WHITE)
- net at R141.2: now also LED45.2 (GREEN), LED49.2 (GREEN), LED53.2 (GREEN), LED57.2 (GREEN), LED61.2 (GREEN), LED65.2 (GREEN), LED69.2 (GREEN), LED73.2 (GREEN), LED77.2 (GREEN), LED81.2 (GREEN)
- no-connect marks 0 -> 2
Other:
- note added: "Unused channels. Consider for indicators"
- note removed: "In the next verision I can do we'll cascade IS31FL3733 and IS31FL3737 drivers"
- note removed: "The matrix I've layed out thus far is too small.Should be double the size."
- moved on the sheet: LED10, LED11, LED12, LED13, LED14, LED15, LED16, LED17, LED18, LED19, LED1_1, LED20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

Commit message: feat(v1 hardware): clean up led matrix
Parts:
- renumbered LED10 to LED10_1, LED52 to LED10_2, LED11 to LED11_1, LED53 to LED11_2, LED12 to LED12_1, LED54 to LED12_2, LED13 to LED13_1, LED55 to LED13_2, LED14 to LED14_1, LED56 to LED14_2, LED15 to LED15_1, LED57 to LED15_2, LED16 to LED16_1, LED58 to LED16_2, LED17 to LED17_1, LED59 to LED17_2, LED18 to LED18_1, LED60 to LED18_2, LED19 to LED19_1, LED61 to LED19_2, LED43 to LED1_2, LED20 to LED20_1, LED62 to LED20_2, LED21 to LED21_1, LED63 to LED21_2, LED22 to LED22_1, LED64 to LED22_2, LED23 to LED23_1, LED65 to LED23_2, LED24 to LED24_1, LED66 to LED24_2, LED25 to LED25_1, LED67 to LED25_2, LED26 to LED26_1, LED68 to LED26_2, LED27 to LED27_1, LED69 to LED27_2, LED28 to LED28_1, LED70 to LED28_2, LED29 to LED29_1, LED71 to LED29_2, LED44 to LED2_2, LED30 to LED30_1, LED72 to LED30_2, LED31 to LED31_1, LED73 to LED31_2, LED32 to LED32_1, LED74 to LED32_2, LED33 to LED33_1, LED75 to LED33_2, LED34 to LED34_1, LED76 to LED34_2, LED35 to LED35_1, LED77 to LED35_2, LED36 to LED36_1, LED78 to LED36_2, LED37 to LED37_1, LED79 to LED37_2, LED38 to LED38_1, LED80 to LED38_2, LED39 to LED39_1, LED81 to LED39_2, LED45 to LED3_2, LED40 to LED40_1, LED82 to LED40_2, LED41 to LED41_1, LED83 to LED41_2, LED42 to LED42_1, LED84 to LED42_2, LED4 to LED4_1, LED46 to LED4_2, LED5 to LED5_1, LED47 to LED5_2, LED6 to LED6_1, LED48 to LED6_2, LED7 to LED7_1, LED49 to LED7_2, LED8 to LED8_1, LED50 to LED8_2, LED9 to LED9_1, LED51 to LED9_2
