File: hardware/v1-electronics/led_matrix.kicad_sch (KiCad schematic)
At the start: 116 parts

Commit message: fix(v1 hardware): fixed the matrix circuit
the change in LED Matrix Driver results in a need to change how we
wire the matrix. this diff accounts for that.

i needed to use a script to rename labels.
Parts:
- removed R119, R120, R121, R122, R123, R124, R125, R126, R127, R128, R129, R130, R131, R132, R133, R134, R135, R136, R137, R138, R139, R140, R141, R142, R143, R144, R145, R146, R147, R177, R67, R69: R_Small, symbol Device:R_Small
Connections:
- net SW5_B_2: now reaches LED17_2.1 (BLUE)
- net SW5_B_2: now also LED18_2.1 (BLUE), LED19_2.1 (BLUE), LED20_2.1 (BLUE), LED21_2.1 (BLUE), LED22_2.1 (BLUE), LED23_2.1 (BLUE), LED24_2.1 (BLUE), LED25_2.1 (BLUE), LED26_2.1 (BLUE), LED27_2.1 (BLUE), LED28_2.1 (BLUE), LED29_2.1 (BLUE), LED30_2.1 (BLUE), LED31_2.1 (BLUE), LED32_2.1 (BLUE)
- net SW6_G_2: now reaches LED17_2.2 (GREEN)
- net SW6_G_2: now also LED18_2.2 (GREEN), LED19_2.2 (GREEN), LED20_2.2 (GREEN), LED21_2.2 (GREEN), LED22_2.2 (GREEN), LED23_2.2 (GREEN), LED24_2.2 (GREEN), LED25_2.2 (GREEN), LED26_2.2 (GREEN), LED27_2.2 (GREEN), LED28_2.2 (GREEN), LED29_2.2 (GREEN), LED30_2.2 (GREEN), LED31_2.2 (GREEN), LED32_2.2 (GREEN)
- net SW7_R_2: now reaches LED17_2.3 (RED)
- net SW7_R_2: now also LED18_2.3 (RED), LED19_2.3 (RED), LED20_2.3 (RED), LED21_2.3 (RED), LED22_2.3 (RED), LED23_2.3 (RED), LED24_2.3 (RED), LED25_2.3 (RED), LED26_2.3 (RED), LED27_2.3 (RED), LED28_2.3 (RED), LED29_2.3 (RED), LED30_2.3 (RED), LED31_2.3 (RED), LED32_2.3 (RED)
- net SW8_W_2: now reaches LED17_2.4 (WHITE)
- net SW8_W_2: now also LED18_2.4 (WHITE), LED19_2.4 (WHITE), LED20_2.4 (WHITE), LED21_2.4 (WHITE), LED22_2.4 (WHITE), LED23_2.4 (WHITE), LED24_2.4 (WHITE), LED25_2.4 (WHITE), LED26_2.4 (WHITE), LED27_2.4 (WHITE), LED28_2.4 (WHITE), LED29_2.4 (WHITE), LED30_2.4 (WHITE), LED31_2.4 (WHITE), LED32_2.4 (WHITE)
- removed net SW10_1: LED37_1.5 (ANODE), LED38_1.5 (ANODE), LED39_1.5 (ANODE), LED40_1.5 (ANODE)
- removed net SW10_2: LED37_2.5 (ANODE), LED38_2.5 (ANODE), LED39_2.5 (ANODE), LED40_2.5 (ANODE)
- net SW11_1 renamed CS10_1
- net CS10_1: now also LED10_1.5 (ANODE), LED26_1.5 (ANODE); no longer LED41_1.5 (ANODE)
- net SW11_2 renamed CS10_2
- net CS10_2: now also LED10_2.5 (ANODE), LED26_2.5 (ANODE); no longer LED41_2.5 (ANODE)
- removed net SW1_1: LED1_1.5 (ANODE), LED2_1.5 (ANODE), LED3_1.5 (ANODE), LED4_1.5 (ANODE)
- removed net SW1_2: LED1_2.5 (ANODE), LED2_2.5 (ANODE), LED3_2.5 (ANODE), LED4_2.5 (ANODE)
- removed net SW2_1: LED5_1.5 (ANODE), LED6_1.5 (ANODE), LED7_1.5 (ANODE), LED8_1.5 (ANODE)
- removed net SW2_2: LED5_2.5 (ANODE), LED6_2.5 (ANODE), LED7_2.5 (ANODE), LED8_2.5 (ANODE)
- removed net SW3_1: LED10_1.5 (ANODE), LED11_1.5 (ANODE), LED12_1.5 (ANODE), LED9_1.5 (ANODE)
- removed net SW3_2: LED10_2.5 (ANODE), LED11_2.5 (ANODE), LED12_2.5 (ANODE), LED9_2.5 (ANODE)
- removed net SW4_1: LED13_1.5 (ANODE), LED14_1.5 (ANODE), LED15_1.5 (ANODE), LED16_1.5 (ANODE)
- removed net SW4_2: LED13_2.5 (ANODE), LED14_2.5 (ANODE), LED15_2.5 (ANODE), LED16_2.5 (ANODE)
- removed net SW5_1: LED17_1.5 (ANODE), LED18_1.5 (ANODE), LED19_1.5 (ANODE), LED20_1.5 (ANODE)
- removed net SW5_2: LED17_2.5 (ANODE), LED18_2.5 (ANODE), LED19_2.5 (ANODE), LED20_2.5 (ANODE)
- removed net SW6_1: LED21_1.5 (ANODE), LED22_1.5 (ANODE), LED23_1.5 (ANODE), LED24_1.5 (ANODE)
- removed net SW6_2: LED21_2.5 (ANODE), LED22_2.5 (ANODE), LED23_2.5 (ANODE), LED24_2.5 (ANODE)
- removed net SW7_1: LED25_1.5 (ANODE), LED26_1.5 (ANODE), LED27_1.5 (ANODE), LED28_1.5 (ANODE)
- removed net SW7_2: LED25_2.5 (ANODE), LED26_2.5 (ANODE), LED27_2.5 (ANODE), LED28_2.5 (ANODE)
- removed net SW8_1: LED29_1.5 (ANODE), LED30_1.5 (ANODE), LED31_1.5 (ANODE), LED32_1.5 (ANODE)
- removed net SW8_2: LED29_2.5 (ANODE), LED30_2.5 (ANODE), LED31_2.5 (ANODE), LED32_2.5 (ANODE)
- removed net SW9_1: LED33_1.5 (ANODE), LED34_1.5 (ANODE), LED35_1.5 (ANODE), LED36_1.5 (ANODE)
- removed net SW9_2: LED33_2.5 (ANODE), LED34_2.5 (ANODE), LED35_2.5 (ANODE), LED36_2.5 (ANODE)
- new net CS11_1: LED11_1.5 (ANODE), LED27_1.5 (ANODE)
- new net CS11_2: LED11_2.5 (ANODE), LED27_2.5 (ANODE)
- new net CS12_1: LED12_1.5 (ANODE), LED28_1.5 (ANODE)
- new net CS12_2: LED12_2.5 (ANODE), LED28_2.5 (ANODE)
- new net CS13_1: LED13_1.5 (ANODE), LED29_1.5 (ANODE)
- new net CS13_2: LED13_2.5 (ANODE), LED29_2.5 (ANODE)
- new net CS14_1: LED14_1.5 (ANODE), LED30_1.5 (ANODE)
- new net CS14_2: LED14_2.5 (ANODE), LED30_2.5 (ANODE)
- new net CS15_1: LED15_1.5 (ANODE), LED31_1.5 (ANODE)
- new net CS15_2: LED15_2.5 (ANODE), LED31_2.5 (ANODE)
- new net CS16_1: LED16_1.5 (ANODE), LED32_1.5 (ANODE)
- new net CS16_2: LED16_2.5 (ANODE), LED32_2.5 (ANODE)
- new net CS1_1: LED17_1.5 (ANODE), LED1_1.5 (ANODE), LED33_1.5 (ANODE)
- new net CS1_2: LED17_2.5 (ANODE), LED1_2.5 (ANODE), LED33_2.5 (ANODE)
- new net CS2_1: LED18_1.5 (ANODE), LED2_1.5 (ANODE), LED34_1.5 (ANODE)
- new net CS2_2: LED18_2.5 (ANODE), LED2_2.5 (ANODE), LED34_2.5 (ANODE)
- new net CS3_1: LED19_1.5 (ANODE), LED35_1.5 (ANODE), LED3_1.5 (ANODE)
- new net CS3_2: LED19_2.5 (ANODE), LED35_2.5 (ANODE), LED3_2.5 (ANODE)
- new net CS4_1: LED20_1.5 (ANODE), LED36_1.5 (ANODE), LED4_1.5 (ANODE)
- new net CS4_2: LED20_2.5 (ANODE), LED36_2.5 (ANODE), LED4_2.5 (ANODE)
- new net CS5_1: LED21_1.5 (ANODE), LED37_1.5 (ANODE), LED5_1.5 (ANODE)
- new net CS5_2: LED21_2.5 (ANODE), LED37_2.5 (ANODE), LED5_2.5 (ANODE)
- new net CS6_1: LED22_1.5 (ANODE), LED38_1.5 (ANODE), LED6_1.5 (ANODE)
- new net CS6_2: LED22_2.5 (ANODE), LED38_2.5 (ANODE), LED6_2.5 (ANODE)
- new net CS7_1: LED23_1.5 (ANODE), LED39_1.5 (ANODE), LED7_1.5 (ANODE)
- new net CS7_2: LED23_2.5 (ANODE), LED39_2.5 (ANODE), LED7_2.5 (ANODE)
- new net CS8_1: LED24_1.5 (ANODE), LED40_1.5 (ANODE), LED8_1.5 (ANODE)
- new net CS8_2: LED24_2.5 (ANODE), LED40_2.5 (ANODE), LED8_2.5 (ANODE)
- new net CS9_1: LED25_1.5 (ANODE), LED41_1.5 (ANODE), LED9_1.5 (ANODE)
- new net CS9_2: LED25_2.5 (ANODE), LED41_2.5 (ANODE), LED9_2.5 (ANODE)
- new net SW10_G_1: LED33_1.2 (GREEN), LED34_1.2 (GREEN), LED35_1.2 (GREEN), LED36_1.2 (GREEN), LED37_1.2 (GREEN), LED38_1.2 (GREEN), LED39_1.2 (GREEN), LED40_1.2 (GREEN), LED41_1.2 (GREEN), LED42_1.2 (GREEN)
- new net SW10_G_2: LED33_2.2 (GREEN), LED34_2.2 (GREEN), LED35_2.2 (GREEN), LED36_2.2 (GREEN), LED37_2.2 (GREEN), LED38_2.2 (GREEN), LED39_2.2 (GREEN), LED40_2.2 (GREEN), LED41_2.2 (GREEN), LED42_2.2 (GREEN)
- new net SW11_R_1: LED33_1.3 (RED), LED34_1.3 (RED), LED35_1.3 (RED), LED36_1.3 (RED), LED37_1.3 (RED), LED38_1.3 (RED), LED39_1.3 (RED), LED40_1.3 (RED), LED41_1.3 (RED), LED42_1.3 (RED)
- new net SW11_R_2: LED33_2.3 (RED), LED34_2.3 (RED), LED35_2.3 (RED), LED36_2.3 (RED), LED37_2.3 (RED), LED38_2.3 (RED), LED39_2.3 (RED), LED40_2.3 (RED), LED41_2.3 (RED), LED42_2.3 (RED)
- new net SW12_W_1: LED33_1.4 (WHITE), LED34_1.4 (WHITE), LED35_1.4 (WHITE), LED36_1.4 (WHITE), LED37_1.4 (WHITE), LED38_1.4 (WHITE), LED39_1.4 (WHITE), LED40_1.4 (WHITE), LED41_1.4 (WHITE), LED42_1.4 (WHITE)
- new net SW12_W_2: LED33_2.4 (WHITE), LED34_2.4 (WHITE), LED35_2.4 (WHITE), LED36_2.4 (WHITE), LED37_2.4 (WHITE), LED38_2.4 (WHITE), LED39_2.4 (WHITE), LED40_2.4 (WHITE), LED41_2.4 (WHITE), LED42_2.4 (WHITE)
- new net SW1_B_1: LED10_1.1 (BLUE), LED11_1.1 (BLUE), LED12_1.1 (BLUE), LED13_1.1 (BLUE), LED14_1.1 (BLUE), LED15_1.1 (BLUE), LED16_1.1 (BLUE), LED1_1.1 (BLUE), LED2_1.1 (BLUE), LED3_1.1 (BLUE), LED4_1.1 (BLUE), LED5_1.1 (BLUE), LED6_1.1 (BLUE), LED7_1.1 (BLUE), LED8_1.1 (BLUE), LED9_1.1 (BLUE)
- new net SW1_B_2: LED10_2.1 (BLUE), LED11_2.1 (BLUE), LED12_2.1 (BLUE), LED13_2.1 (BLUE), LED14_2.1 (BLUE), LED15_2.1 (BLUE), LED16_2.1 (BLUE), LED1_2.1 (BLUE), LED2_2.1 (BLUE), LED3_2.1 (BLUE), LED4_2.1 (BLUE), LED5_2.1 (BLUE), LED6_2.1 (BLUE), LED7_2.1 (BLUE), LED8_2.1 (BLUE), LED9_2.1 (BLUE)
- new net SW2_G_1: LED10_1.2 (GREEN), LED11_1.2 (GREEN), LED12_1.2 (GREEN), LED13_1.2 (GREEN), LED14_1.2 (GREEN), LED15_1.2 (GREEN), LED16_1.2 (GREEN), LED1_1.2 (GREEN), LED2_1.2 (GREEN), LED3_1.2 (GREEN), LED4_1.2 (GREEN), LED5_1.2 (GREEN), LED6_1.2 (GREEN), LED7_1.2 (GREEN), LED8_1.2 (GREEN), LED9_1.2 (GREEN)
- new net SW2_G_2: LED10_2.2 (GREEN), LED11_2.2 (GREEN), LED12_2.2 (GREEN), LED13_2.2 (GREEN), LED14_2.2 (GREEN), LED15_2.2 (GREEN), LED16_2.2 (GREEN), LED1_2.2 (GREEN), LED2_2.2 (GREEN), LED3_2.2 (GREEN), LED4_2.2 (GREEN), LED5_2.2 (GREEN), LED6_2.2 (GREEN), LED7_2.2 (GREEN), LED8_2.2 (GREEN), LED9_2.2 (GREEN)
- new net SW3_R_1: LED10_1.3 (RED), LED11_1.3 (RED), LED12_1.3 (RED), LED13_1.3 (RED), LED14_1.3 (RED), LED15_1.3 (RED), LED16_1.3 (RED), LED1_1.3 (RED), LED2_1.3 (RED), LED3_1.3 (RED), LED4_1.3 (RED), LED5_1.3 (RED), LED6_1.3 (RED), LED7_1.3 (RED), LED8_1.3 (RED), LED9_1.3 (RED)
- new net SW3_R_2: LED10_2.3 (RED), LED11_2.3 (RED), LED12_2.3 (RED), LED13_2.3 (RED), LED14_2.3 (RED), LED15_2.3 (RED), LED16_2.3 (RED), LED1_2.3 (RED), LED2_2.3 (RED), LED3_2.3 (RED), LED4_2.3 (RED), LED5_2.3 (RED), LED6_2.3 (RED), LED7_2.3 (RED), LED8_2.3 (RED), LED9_2.3 (RED)
- new net SW4_W_1: LED10_1.4 (WHITE), LED11_1.4 (WHITE), LED12_1.4 (WHITE), LED13_1.4 (WHITE), LED14_1.4 (WHITE), LED15_1.4 (WHITE), LED16_1.4 (WHITE), LED1_1.4 (WHITE), LED2_1.4 (WHITE), LED3_1.4 (WHITE), LED4_1.4 (WHITE), LED5_1.4 (WHITE), LED6_1.4 (WHITE), LED7_1.4 (WHITE), LED8_1.4 (WHITE), LED9_1.4 (WHITE)
- new net SW4_W_2: LED10_2.4 (WHITE), LED11_2.4 (WHITE), LED12_2.4 (WHITE), LED13_2.4 (WHITE), LED14_2.4 (WHITE), LED15_2.4 (WHITE), LED16_2.4 (WHITE), LED1_2.4 (WHITE), LED2_2.4 (WHITE), LED3_2.4 (WHITE), LED4_2.4 (WHITE), LED5_2.4 (WHITE), LED6_2.4 (WHITE), LED7_2.4 (WHITE), LED8_2.4 (WHITE), LED9_2.4 (WHITE)
- new net SW5_B_1: LED17_1.1 (BLUE), LED18_1.1 (BLUE), LED19_1.1 (BLUE), LED20_1.1 (BLUE), LED21_1.1 (BLUE), LED22_1.1 (BLUE), LED23_1.1 (BLUE), LED24_1.1 (BLUE), LED25_1.1 (BLUE), LED26_1.1 (BLUE), LED27_1.1 (BLUE), LED28_1.1 (BLUE), LED29_1.1 (BLUE), LED30_1.1 (BLUE), LED31_1.1 (BLUE), LED32_1.1 (BLUE)
- new net SW6_G_1: LED17_1.2 (GREEN), LED18_1.2 (GREEN), LED19_1.2 (GREEN), LED20_1.2 (GREEN), LED21_1.2 (GREEN), LED22_1.2 (GREEN), LED23_1.2 (GREEN), LED24_1.2 (GREEN), LED25_1.2 (GREEN), LED26_1.2 (GREEN), LED27_1.2 (GREEN), LED28_1.2 (GREEN), LED29_1.2 (GREEN), LED30_1.2 (GREEN), LED31_1.2 (GREEN), LED32_1.2 (GREEN)
- new net SW7_R_1: LED17_1.3 (RED), LED18_1.3 (RED), LED19_1.3 (RED), LED20_1.3 (RED), LED21_1.3 (RED), LED22_1.3 (RED), LED23_1.3 (RED), LED24_1.3 (RED), LED25_1.3 (RED), LED26_1.3 (RED), LED27_1.3 (RED), LED28_1.3 (RED), LED29_1.3 (RED), LED30_1.3 (RED), LED31_1.3 (RED), LED32_1.3 (RED)
- new net SW8_W_1: LED17_1.4 (WHITE), LED18_1.4 (WHITE), LED19_1.4 (WHITE), LED20_1.4 (WHITE), LED21_1.4 (WHITE), LED22_1.4 (WHITE), LED23_1.4 (WHITE), LED24_1.4 (WHITE), LED25_1.4 (WHITE), LED26_1.4 (WHITE), LED27_1.4 (WHITE), LED28_1.4 (WHITE), LED29_1.4 (WHITE), LED30_1.4 (WHITE), LED31_1.4 (WHITE), LED32_1.4 (WHITE)
- new net SW9_B_1: LED33_1.1 (BLUE), LED34_1.1 (BLUE), LED35_1.1 (BLUE), LED36_1.1 (BLUE), LED37_1.1 (BLUE), LED38_1.1 (BLUE), LED39_1.1 (BLUE), LED40_1.1 (BLUE), LED41_1.1 (BLUE), LED42_1.1 (BLUE)
- new net SW9_B_2: LED33_2.1 (BLUE), LED34_2.1 (BLUE), LED35_2.1 (BLUE), LED36_2.1 (BLUE), LED37_2.1 (BLUE), LED38_2.1 (BLUE), LED39_2.1 (BLUE), LED40_2.1 (BLUE), LED41_2.1 (BLUE), LED42_2.1 (BLUE)
- no-connect marks 2 -> 0
Other:
- note removed: "Unused channels. Consider for indicators"

Commit message: refactor(v1 hardware): convert switch matrix to hierarchical pins
made other changes
had claude generate a script for making the convertion
the references for this file still need to be fixed
Other:
- title: (none) -> Slack
Changed lines of the file:
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@@
 	(generator_version "10.0")
 	(paper "User" 1040 355)
+	(title_block
+		(title "Slack")
+		(date "2026-06-17")
+		(rev "A.0.0")
+	)
 	(text "RGBW LED Matrix Halve 2"
 		(exclude_from_sim no)
