File: hardware/v1-electronics/led_matrix.kicad_sch (KiCad schematic)
At the start: 85 parts

Commit message: checkpoint(v1 hardware): this is the save before corrections
Parts:
- added LED501, LED502, LED503, LED504, LED505, LED506, LED507, LED508, LED509, LED510, LED511, LED512: LTST-FC12WEGBD-5A, LTSTFC12WEGBD5A, symbol Lite-On LTST-FC12WEGBD-5A:LTST-FC12WEGBD-5A
Connections:
- net Chip1CurrentSource15: now also LED501.5 (ANODE), LED502.5 (ANODE), LED503.5 (ANODE)
- net Chip1CurrentSource16: now also LED504.5 (ANODE), LED505.5 (ANODE), LED506.5 (ANODE)
- net Chip1SinkSwitch1: now also LED501.1 (BLUE), LED504.1 (BLUE)
- net Chip1SinkSwitch10: now also LED503.2 (GREEN), LED506.2 (GREEN)
- net Chip1SinkSwitch11: now also LED503.3 (RED), LED506.3 (RED)
- net Chip1SinkSwitch12: now also LED503.4 (WHITE), LED506.4 (WHITE)
- net Chip1SinkSwitch2: now also LED501.2 (GREEN), LED504.2 (GREEN)
- net Chip1SinkSwitch3: now also LED501.3 (RED), LED504.3 (RED)
- net Chip1SinkSwitch4: now also LED501.4 (WHITE), LED504.4 (WHITE)
- net Chip1SinkSwitch5: now also LED502.1 (BLUE), LED505.1 (BLUE)
- net Chip1SinkSwitch6: now also LED502.2 (GREEN), LED505.2 (GREEN)
- net Chip1SinkSwitch7: now also LED502.3 (RED), LED505.3 (RED)
- net Chip1SinkSwitch8: now also LED502.4 (WHITE), LED505.4 (WHITE)
- net Chip1SinkSwitch9: now also LED503.1 (BLUE), LED506.1 (BLUE)
- net Chip2CurrentSource15: now also LED507.5 (ANODE), LED508.5 (ANODE), LED509.5 (ANODE)
- net Chip2CurrentSource16: now also LED510.5 (ANODE), LED511.5 (ANODE), LED512.5 (ANODE)
- net Chip2SinkSwitch1: now also LED507.1 (BLUE), LED510.1 (BLUE)
- net Chip2SinkSwitch10: now also LED509.2 (GREEN), LED512.2 (GREEN)
- net Chip2SinkSwitch11: now also LED509.3 (RED), LED512.3 (RED)
- net Chip2SinkSwitch12: now also LED509.4 (WHITE), LED512.4 (WHITE)
- net Chip2SinkSwitch2: now also LED507.2 (GREEN), LED510.2 (GREEN)
- net Chip2SinkSwitch3: now also LED507.3 (RED), LED510.3 (RED)
- net Chip2SinkSwitch4: now also LED507.4 (WHITE), LED510.4 (WHITE)
- net Chip2SinkSwitch5: now also LED508.1 (BLUE), LED511.1 (BLUE)
- net Chip2SinkSwitch6: now also LED508.2 (GREEN), LED511.2 (GREEN)
- net Chip2SinkSwitch7: now also LED508.3 (RED), LED511.3 (RED)
- net Chip2SinkSwitch8: now also LED508.4 (WHITE), LED511.4 (WHITE)
- net Chip2SinkSwitch9: now also LED509.1 (BLUE), LED512.1 (BLUE)
- no-connect marks 28 -> 24
Other:
- note added: "Indicators"

Commit message: fix(v1 hardware): complete set of recommendations
Other:
- sheet LED Matrix Controller 1 ports: added ~{Interrupt}; removed Interrupt
- sheet LED Matrix Controller 2 ports: added ~{Interrupt}; removed Interrupt
Changed lines of the file:
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@@
 		)
 	)
-	(hierarchical_label "Chip1Interrupt"
+	(hierarchical_label "~{Chip1Interrupt}"
 		(shape input)
 		(at 81.28 76.2 0)
@@
 		)
 	)
-	(hierarchical_label "Chip2Interrupt"
+	(hierarchical_label "~{Chip2Interrupt}"
 		(shape input)
 		(at 81.28 231.14 0)
@@
 			)
 		)
-		(pin "Interrupt" input
+		(pin "~{Interrupt}" input
 			(at 81.28 231.14 0)
 			(effects
@@
 			)
 		)
-		(pin "Interrupt" input
+		(pin "~{Interrupt}" input
 			(at 81.28 76.2 0)
 			(effects

Commit message: feat(v1 hardware): place foot prints
Parts:
- JP1: footprint (none) -> Connector_PinHeader_2.54mm:PinHeader_1x02_P2.54mm_Vertical
