File: hardware/v1-electronics/led_matrix.kicad_sch (KiCad schematic)
At the start: 97 parts

Commit message: feat(v1 hardware): all power train components foot prints selected
Parts:
- LED1, LED10, LED11, LED12, LED13, LED14, LED15, LED16, LED17, LED18, LED19, LED2, LED20, LED21, LED22, LED23, LED24, LED25, LED26, LED27, LED28, LED29, LED3, LED30, LED31, LED32, LED33, LED34, LED35, LED36, LED37, LED38, LED39, LED4, LED40, LED41, LED42, LED43, LED44, LED45, LED46, LED47, LED48, LED49, LED5, LED50, LED501, LED502, LED503, LED504, LED505, LED506, LED507, LED508, LED509, LED51, LED510, LED511, LED512, LED52, LED53, LED54, LED55, LED56, LED57, LED58, LED59, LED6, LED60, LED61, LED62, LED63, LED66, LED67, LED68, LED69, LED7, LED70, LED71, LED72, LED73, LED74, LED75, LED76, LED77, LED78, LED79, LED8, LED80, LED81, LED82, LED83, LED84, LED85, LED86, LED9: footprint LTSTFC12WEGBD5A -> Liteon:LTSTFC12WEGBD5A

Commit message: feat(v1 hardware): transfer to ergogen layout
Parts:
- renumbered LED79 to LED511, LED501 to LED512, LED502 to LED513, LED503 to LED514, LED504 to LED515, LED505 to LED517, LED506 to LED518, LED86 to LED521, LED507 to LED522, LED508 to LED523, LED509 to LED524, LED510 to LED525, LED511 to LED526, LED512 to LED527, LED66 to LED63, LED67 to LED64, LED68 to LED65, LED69 to LED66, LED70 to LED67, LED71 to LED68, LED63 to LED69, LED73 to LED70, LED74 to LED71, LED75 to LED72, LED76 to LED73, LED77 to LED74, LED78 to LED75, LED72 to LED76, LED80 to LED77, LED81 to LED78, LED82 to LED79, LED83 to LED80, LED84 to LED81, LED85 to LED82
Connections:
- net Chip1CurrentSource11: now also LED61.5 (ANODE)

Commit message: feat(v1 hardware): update config switch
Parts:
- JP1: footprint Connector_PinHeader_2.54mm:PinHeader_1x02_P2.54mm_Vertical -> Dongguan Guangzhu Industrial:DSIC01LSGET
Changed lines of the file:
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@@
 			)
 		)
-		(property "Footprint" "Connector_PinHeader_2.54mm:PinHeader_1x02_P2.54mm_Vertical"
+		(property "Footprint" "Dongguan Guangzhu Industrial:DSIC01LSGET"
 			(at 101.6 111.76 0)
 			(hide yes)
