File: hardware/v1-electronics/matric_controller_1.kicad_sch (KiCad schematic)
At the start: 13 parts, among them IC1 IS31FL3733-QFLS4-TR

Commit message: refactor(v1 hardware): get references in order
Parts:
- renumbered C25 to C21, C33 to C22, C37 to C23, C35 to C24, C38 to C25, C36 to C34, C39 to C35, C24 to C36, IC1 to IC3, R114 to R41, R103 to R42, R113 to R43, R102 to R44
Connections:
- net Chip1CurrentSource1 renamed CurrentSource1
- net Chip1CurrentSource10 renamed CurrentSource10
- net Chip1CurrentSource11 renamed CurrentSource11
- net Chip1CurrentSource12 renamed CurrentSource12
- net Chip1CurrentSource13 renamed CurrentSource13
- net Chip1CurrentSource14 renamed CurrentSource14
- net Chip1CurrentSource15 renamed CurrentSource15
- net Chip1CurrentSource16 renamed CurrentSource16
- net Chip1CurrentSource2 renamed CurrentSource2
- net Chip1CurrentSource3 renamed CurrentSource3
- net Chip1CurrentSource4 renamed CurrentSource4
- net Chip1CurrentSource5 renamed CurrentSource5
- net Chip1CurrentSource6 renamed CurrentSource6
- net Chip1CurrentSource7 renamed CurrentSource7
- net Chip1CurrentSource8 renamed CurrentSource8
- net Chip1CurrentSource9 renamed CurrentSource9
- net Chip1SinkSwitch1 renamed SinkSwitch1
- net Chip1SinkSwitch10 renamed SinkSwitch10
- net Chip1SinkSwitch11 renamed SinkSwitch11
- net Chip1SinkSwitch12 renamed SinkSwitch12
- net Chip1SinkSwitch2 renamed SinkSwitch2
- net Chip1SinkSwitch3 renamed SinkSwitch3
- net Chip1SinkSwitch4 renamed SinkSwitch4
- net Chip1SinkSwitch5 renamed SinkSwitch5
- net Chip1SinkSwitch6 renamed SinkSwitch6
- net Chip1SinkSwitch7 renamed SinkSwitch7
- net Chip1SinkSwitch8 renamed SinkSwitch8
- net Chip1SinkSwitch9 renamed SinkSwitch9
Other:
- note removed: "I2C Manual Reset"
- moved on the sheet: C36, R42, R43, R44
