File: hardware/v1-electronics/matric_controller_1.kicad_sch (KiCad schematic)
At the start: 13 parts, among them IC3 IS31FL3733-QFLS4-TR

Commit message: checkpoint(v1 hardware): this is the save before corrections
Connections:
- net VDD renamed V_REG0
- net V_SYS renamed +5V
Other:
- title: (none) -> Slack
Changed lines of the file:
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@@
 	(generator_version "10.0")
 	(paper "A")
+	(title_block
+		(title "Slack")
+		(date "2026-07-12")
+		(rev "A.0.3")
+	)
 	(rectangle
 		(start 15.24 91.44)
@@
 		)
 	)
-	(text_box "This circuit is incomplete:\n- SDB shuts the ic down when pulled low, why is it pulled low on the schematic?"
-		(exclude_from_sim no)
-		(at 121.92 193.04 0)
-		(size 38.1 10.1599)
-		(margins 0.9525 0.9525 0.9525 0.9525)
-		(stroke
-			(width 0)
-			(type solid)
-		)
-		(fill
-			(type color)
-			(color 255 229 191 1)
-		)
-		(effects
-			(font
-				(size 1.27 1.27)
-			)
-			(justify left top)
-		)
-	)
 	(junction
 		(at 73.66 55.88)
@@
 		(dnp no)
 		(property "Reference" "IC3"
-			(at 231.14 45.72 0)
+			(at 218.44 43.18 0)
 			(show_name no)
 			(do_not_autoplace no)
@@
 					(size 1.27 1.27)
 				)
+				(justify left top)
 			)
 		)
 		(property "Value" "IS31FL3733-QFLS4-TR"
-			(at 231.14 48.26 0)
+			(at 218.44 45.72 0)
 			(show_name no)
 			(do_not_autoplace no)
@@
 					(size 1.27 1.27)
 				)
+				(justify left top)
 			)
 		)
@@
 			)
 		)
-		(property "Value" "V_SYS"
+		(property "Value" "+5V"
 			(at 58.42 30.48 0)
 			(show_name no)
@@
 			)
 		)
-		(property "Value" "VDD"
+		(property "Value" "V_REG0"
 			(at 88.9 101.6 0)
 			(show_name no)
@@
 			)
 		)
-		(property "Value" "VDD"
+		(property "Value" "V_REG0"
 			(at 53.34 132.08 0)
 			(show_name no)

Commit message: fix(v1 hardware): complete set of recommendations
Parts:
- removed R44: 100kΩ, symbol Device:R_Small
Connections:
- net Interrupt renamed ~{Interrupt}
Other:
- moved on the sheet: R42, R43

Commit message: feat(v1 hardware): place foot prints
Parts:
- C21: footprint (none) -> Capacitor_Tantalum_SMD:CP_EIA-3216-18_Kemet-A; symbol Device:C_Small_US -> Device:C_Polarized_Small
- C22, C24, C34, C36: footprint (none) -> Capacitor_SMD:C_0805_2012Metric
- C23, C25, C35: footprint (none) -> Capacitor_SMD:C_0402_1005Metric
- IC3: footprint QFN40P600X600X80-49N-D -> Lumissil Microsystems:QFN40P600X600X80-49N-D
- R41: footprint (none) -> Resistor_SMD:R_0201_0603Metric
- R42, R43: footprint (none) -> Resistor_SMD:R_0805_2012Metric

Commit message: feat(v1 hardware): review fixes
Parts:
- R41: value 13kΩ -> 22kΩ
Changed lines of the file:
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@@
 			)
 		)
-		(property "Value" "13kΩ"
+		(property "Value" "22kΩ"
 			(at 30.48 110.4899 0)
 			(show_name no)
@@
 			)
 		)
-		(property "Description" "part selected: 0603WAF1302T5E"
+		(property "Description" "part selected: 0603WAF2202T5E"
 			(at 27.94 109.22 0)
 			(hide yes)
