File: hardware/v1-electronics/matrix_controller_2.kicad_sch (KiCad schematic)
At the start: 13 parts, among them IC2 IS31FL3733-QFLS4-TR

Commit message: refactor(v1 hardware): get references in order
Parts:
- removed R106, R107, R118: 100kΩ, symbol Device:R_Small
- added R46, R47, R48: 100kΩ, symbol Device:R_Small
- renumbered C40 to C27, C43 to C28, C41 to C29, C44 to C30, C42 to C31, C45 to C32, C28 to C33, IC2 to IC4, R117 to R45
Connections:
- net DGND: now also R46.1, R47.1
- net I2C_Reset: now also R47.2
- net Interrupt: now also R48.2
- net Shutdown: now also R46.2
- net VDD: now also R48.1
- net Chip2CurrentSource1 renamed CurrentSource1
- net Chip2CurrentSource10 renamed CurrentSource10
- net Chip2CurrentSource11 renamed CurrentSource11
- net Chip2CurrentSource12 renamed CurrentSource12
- net Chip2CurrentSource13 renamed CurrentSource13
- net Chip2CurrentSource14 renamed CurrentSource14
- net Chip2CurrentSource15 renamed CurrentSource15
- net Chip2CurrentSource16 renamed CurrentSource16
- net Chip2CurrentSource2 renamed CurrentSource2
- net Chip2CurrentSource3 renamed CurrentSource3
- net Chip2CurrentSource4 renamed CurrentSource4
- net Chip2CurrentSource5 renamed CurrentSource5
- net Chip2CurrentSource6 renamed CurrentSource6
- net Chip2CurrentSource7 renamed CurrentSource7
- net Chip2CurrentSource8 renamed CurrentSource8
- net Chip2CurrentSource9 renamed CurrentSource9
- net Chip2SinkSwitch1 renamed SinkSwitch1
- net Chip2SinkSwitch10 renamed SinkSwitch10
- net Chip2SinkSwitch11 renamed SinkSwitch11
- net Chip2SinkSwitch12 renamed SinkSwitch12
- net Chip2SinkSwitch2 renamed SinkSwitch2
- net Chip2SinkSwitch3 renamed SinkSwitch3
- net Chip2SinkSwitch4 renamed SinkSwitch4
- net Chip2SinkSwitch5 renamed SinkSwitch5
- net Chip2SinkSwitch6 renamed SinkSwitch6
- net Chip2SinkSwitch7 renamed SinkSwitch7
- net Chip2SinkSwitch8 renamed SinkSwitch8
- net Chip2SinkSwitch9 renamed SinkSwitch9
Other:
- note removed: "I2C Manual Reset"
- moved on the sheet: C33
