File: hardware/v1-electronics/switch_matrix.kicad_sch (KiCad schematic)
At the start: 230 parts, among them SW1 MSwitch, SW10 MSwitch, SW11 MSwitch, SW12 MSwitch, SW13 MSwitch, SW14 MSwitch, SW15 MSwitch, SW16 MSwitch, SW17 MSwitch, SW18 MSwitch, SW19 MSwitch, SW2 MSwitch, SW20 MSwitch, SW23 MSwitch, SW24 MSwitch, SW25 MSwitch, SW26 MSwitch, SW27 MSwitch, SW28 MSwitch, SW29 MSwitch, SW3 MSwitch, SW30 MSwitch, SW31 MSwitch, SW32 MSwitch, SW33 MSwitch, SW34 MSwitch, SW37 MSwitch, SW38 MSwitch, SW39 MSwitch, SW4 MSwitch, SW40 MSwitch, SW41 MSwitch, SW42 MSwitch, SW43 MSwitch, SW44 MSwitch, SW45 MSwitch, SW46 MSwitch, SW47 MSwitch, SW48 MSwitch, SW5 MSwitch, SW51 MSwitch, SW52 MSwitch, SW53 MSwitch, SW54 MSwitch, SW55 MSwitch, SW56 MSwitch, SW57 MSwitch, SW58 MSwitch, SW59 MSwitch, SW6 MSwitch, SW60 MSwitch, SW61 MSwitch, SW62 MSwitch, SW63 SW_Push, SW66 SW_Push, SW67 MSwitch, SW68 MSwitch, SW69 MSwitch, SW70 MSwitch, SW71 MSwitch, SW72 MSwitch, SW73 SW_DIP_x01, SW74 SW_DIP_x01, SW75 SW_DIP_x01, SW76 SW_DIP_x01, SW77 SW_DIP_x01, SW78 SW_DIP_x01, SW79 SW_DIP_x01, SW80 SW_DIP_x01, SW81 SW_DIP_x01, SW82 SW_DIP_x01, SW83 SW_DIP_x01, SW84 SW_DIP_x01, SW85 SW_DIP_x01, SW86 SW_DIP_x01, SW9 MSwitch

Commit message: checkpoint(v1 hardware): this is the save before corrections
Parts:
- renumbered D76 to D86
Connections:
- net VDD renamed V_REG0
Other:
- moved on the sheet: C1, C10, C11, C12, C13, C14, C15, C16, C17, C18, C19, C2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

Commit message: feat(v1 hardware): place foot prints
Parts:
- C1, C10, C11, C12, C13, C14, C15, C16, C17, C18, C19, C2, C20, C3, C4, C5, C6, C7, C8, C9: footprint (none) -> Capacitor_SMD:C_0402_1005Metric
- D1, D10, D11, D12, D13, D14, D15, D16, D17, D18, D19, D2, D20, D21, D22, D23, D24, D25, D26, D27, D28, D29, D3, D30, D31, D32, D33, D34, D35, D36, D37, D38, D39, D4, D40, D41, D42, D43, D44, D45, D46, D47, D48, D49, D5, D50, D51, D52, D53, D54, D55, D56, D57, D58, D59, D6, D60, D61, D62, D63, D66, D67, D68, D69, D7, D70, D71, D72, D73, D74, D75, D76, D77, D78, D79, D8, D80, D81, D82, D83, D84, D85, D86, D9: footprint (none) -> Diode_SMD:D_SOD-523
- R1, R10, R11, R12, R13, R14, R15, R16, R17, R18, R19, R2, R20, R21, R22, R23, R24, R25, R26, R27, R28, R29, R3, R30, R31, R32, R33, R34, R35, R36, R37, R38, R39, R4, R40, R5, R6, R7, R8, R9: footprint (none) -> Resistor_SMD:R_0805_2012Metric
- RE1/SW7, RE2/SW8, RE3/SW21, RE4/SW22, RE5/SW35, RE6/SW36, RE7/SW49, RE8/SW50: footprint (none) -> ALPS Electric:EC09E1524418
- RE10, RE9: footprint (none) -> ALPS Electric:EC10E1220505
- SW1, SW10, SW11, SW12, SW13, SW14, SW15, SW16, SW17, SW18, SW19, SW2, SW20, SW23, SW24, SW25, SW26, SW27, SW28, SW29, SW3, SW30, SW31, SW32, SW33, SW34, SW37, SW38, SW39, SW4, SW40, SW41, SW42, SW43, SW44, SW45, SW46, SW47, SW48, SW5, SW51, SW52, SW53, SW54, SW55, SW56, SW57, SW58, SW59, SW6, SW60, SW61, SW62, SW67, SW68, SW69, SW70, SW71, SW72, SW9: footprint (none) -> Cherry:Cherry_ULP_SMD
- SW63, SW66: footprint (none) -> Button_Switch_SMD:SW_Push_1P1T_XKB_TS-1187A

Commit message: feat(v1 hardware): all power train components foot prints selected
Parts:
- RE1/SW7, RE2/SW8, RE3/SW21, RE4/SW22, RE5/SW35, RE6/SW36, RE7/SW49, RE8/SW50: footprint ALPS Electric:EC09E1524418 -> Bourns:PEC11S929KS0015
Changed lines of the file:
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@@
 			)
 		)
-		(property "Footprint" "ALPS Electric:EC09E1524418"
+		(property "Footprint" "Bourns:PEC11S929KS0015"
 			(at 430.53 87.376 0)
 			(hide yes)
@@
 			)
 		)
-		(property "Description" "part selected: EC09E1524418"
+		(property "Description" "part selected: PEC11S929KS0015"
 			(at 434.34 91.44 0)
 			(hide yes)
@@
 			)
 		)
-		(property "Footprint" "ALPS Electric:EC09E1524418"
+		(property "Footprint" "Bourns:PEC11S929KS0015"
 			(at 222.25 197.104 0)
 			(hide yes)
@@
 			)
 		)
-		(property "Description" "part selected: EC09E1524418"
+		(property "Description" "part selected: PEC11S929KS0015"
 			(at 218.44 193.04 0)
 			(hide yes)
@@
 			)
 		)
-		(property "Footprint" "ALPS Electric:EC09E1524418"
+		(property "Footprint" "Bourns:PEC11S929KS0015"
 			(at 430.53 36.576 0)
 			(hide yes)
@@
 			)
 		)
-		(property "Description" "part selected: EC09E1524418"
+		(property "Description" "part selected: PEC11S929KS0015"
 			(at 434.34 40.64 0)
 			(hide yes)
@@
 			)
 		)
-		(property "Footprint" "ALPS Electric:EC09E1524418"
+		(property "Footprint" "Bourns:PEC11S929KS0015"
 			(at 430.53 188.976 0)
 			(hide yes)
@@
 			)
 		)
-		(property "Description" "part selected: EC09E1524418"
+		(property "Description" "part selected: PEC11S929KS0015"
 			(at 434.34 193.04 0)
 			(hide yes)
@@
 			)
 		)
-		(property "Footprint" "ALPS Electric:EC09E1524418"
+		(property "Footprint" "Bourns:PEC11S929KS0015"
 			(at 222.25 95.504 0)
 			(hide yes)
@@
 			)
 		)
-		(property "Description" "part selected: EC09E1524418"
+		(property "Description" "part selected: PEC11S929KS0015"
 			(at 218.44 91.44 0)
 			(hide yes)
@@
 			)
 		)
-		(property "Footprint" "ALPS Electric:EC09E1524418"
+		(property "Footprint" "Bourns:PEC11S929KS0015"
 			(at 222.25 44.704 0)
 			(hide yes)
@@
 			)
 		)
-		(property "Description" "part selected: EC09E1524418"
+		(property "Description" "part selected: PEC11S929KS0015"
 			(at 218.44 40.64 0)
 			(hide yes)
@@
 			)
 		)
-		(property "Footprint" "ALPS Electric:EC09E1524418"
+		(property "Footprint" "Bourns:PEC11S929KS0015"
 			(at 430.53 138.176 0)
 			(hide yes)
@@
 			)
 		)
-		(property "Description" "part selected: EC09E1524418"
+		(property "Description" "part selected: PEC11S929KS0015"
 			(at 434.34 142.24 0)
 			(hide yes)
@@
 			)
 		)
-		(property "Footprint" "ALPS Electric:EC09E1524418"
+		(property "Footprint" "Bourns:PEC11S929KS0015"
 			(at 222.25 146.304 0)
 			(hide yes)
@@
 			)
 		)
-		(property "Description" "part selected: EC09E1524418"
+		(property "Description" "part selected: PEC11S929KS0015"
 			(at 218.44 142.24 0)
 			(hide yes)

Commit message: feat(v1 hardware): all components have unrefined footprints
Parts:
- SW73, SW74, SW75, SW76, SW77, SW78, SW79, SW80, SW81, SW82, SW83, SW84, SW85, SW86: footprint (none) -> Amazon:1208YD
Changed lines of the file:
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@@
 			)
 		)
-		(property "Footprint" ""
+		(property "Footprint" "Amazon:1208YD"
 			(at 124.46 304.8 0)
 			(hide yes)
@@
 			)
 		)
-		(property "Footprint" ""
+		(property "Footprint" "Amazon:1208YD"
 			(at 533.4 304.8 0)
 			(hide yes)
@@
 			)
 		)
-		(property "Footprint" ""
+		(property "Footprint" "Amazon:1208YD"
 			(at 96.52 304.8 0)
 			(hide yes)
@@
 			)
 		)
-		(property "Footprint" ""
+		(property "Footprint" "Amazon:1208YD"
 			(at 505.46 304.8 0)
 			(hide yes)
@@
 			)
 		)
-		(property "Footprint" ""
+		(property "Footprint" "Amazon:1208YD"
 			(at 40.64 304.8 0)
 			(hide yes)
@@
 			)
 		)
-		(property "Footprint" ""
+		(property "Footprint" "Amazon:1208YD"
 			(at 617.22 304.8 0)
 			(hide yes)
@@
 			)
 		)
-		(property "Footprint" ""
+		(property "Footprint" "Amazon:1208YD"
 			(at 208.28 304.8 0)
 			(hide yes)
@@
 			)
 		)
-		(property "Footprint" ""
+		(property "Footprint" "Amazon:1208YD"
 			(at 180.34 304.8 0)
 			(hide yes)
@@
 			)
 		)
-		(property "Footprint" ""
+		(property "Footprint" "Amazon:1208YD"
 			(at 561.34 304.8 0)
 			(hide yes)
@@
 			)
 		)
-		(property "Footprint" ""
+		(property "Footprint" "Amazon:1208YD"
 			(at 68.58 304.8 0)
 			(hide yes)
@@
 			)
 		)
-		(property "Footprint" ""
+		(property "Footprint" "Amazon:1208YD"
 			(at 477.52 304.8 0)
 			(hide yes)
@@
 			)
 		)
-		(property "Footprint" ""
+		(property "Footprint" "Amazon:1208YD"
 			(at 589.28 304.8 0)
 			(hide yes)
@@
 			)
 		)
-		(property "Footprint" ""
+		(property "Footprint" "Amazon:1208YD"
 			(at 452.12 304.8 0)
 			(hide yes)
@@
 			)
 		)
-		(property "Footprint" ""
+		(property "Footprint" "Amazon:1208YD"
 			(at 152.4 304.8 0)
 			(hide yes)
