File: hardware/v1-electronics/switch_matrix.kicad_sch (KiCad schematic)
At the start: 230 parts, among them SW1 MSwitch, SW10 MSwitch, SW11 MSwitch, SW12 MSwitch, SW13 MSwitch, SW14 MSwitch, SW15 MSwitch, SW16 MSwitch, SW17 MSwitch, SW18 MSwitch, SW19 MSwitch, SW2 MSwitch, SW20 MSwitch, SW23 MSwitch, SW24 MSwitch, SW25 MSwitch, SW26 MSwitch, SW27 MSwitch, SW28 MSwitch, SW29 MSwitch, SW3 MSwitch, SW30 MSwitch, SW31 MSwitch, SW32 MSwitch, SW33 MSwitch, SW34 MSwitch, SW37 MSwitch, SW38 MSwitch, SW39 MSwitch, SW4 MSwitch, SW40 MSwitch, SW41 MSwitch, SW42 MSwitch, SW43 MSwitch, SW44 MSwitch, SW45 MSwitch, SW46 MSwitch, SW47 MSwitch, SW48 MSwitch, SW5 MSwitch, SW51 MSwitch, SW52 MSwitch, SW53 MSwitch, SW54 MSwitch, SW55 MSwitch, SW56 MSwitch, SW57 MSwitch, SW58 MSwitch, SW59 MSwitch, SW6 MSwitch, SW60 MSwitch, SW61 MSwitch, SW62 MSwitch, SW63 SW_Push, SW66 SW_Push, SW67 MSwitch, SW68 MSwitch, SW69 MSwitch, SW70 MSwitch, SW71 MSwitch, SW72 MSwitch, SW73 SW_DIP_x01, SW74 SW_DIP_x01, SW75 SW_DIP_x01, SW76 SW_DIP_x01, SW77 SW_DIP_x01, SW78 SW_DIP_x01, SW79 SW_DIP_x01, SW80 SW_DIP_x01, SW81 SW_DIP_x01, SW82 SW_DIP_x01, SW83 SW_DIP_x01, SW84 SW_DIP_x01, SW85 SW_DIP_x01, SW86 SW_DIP_x01, SW9 MSwitch

Commit message: feat(v1 hardware): add all components
Parts:
- SW63, SW66: footprint Button_Switch_SMD:SW_Push_1P1T_XKB_TS-1187A -> XKB Connection:TC-1109-C-E
Changed lines of the file:
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@@
 			)
 		)
-		(property "Footprint" "Button_Switch_SMD:SW_Push_1P1T_XKB_TS-1187A"
+		(property "Footprint" "XKB Connection:TC-1109-C-E"
 			(at 205.74 241.3 0)
 			(hide yes)
@@
 			)
 		)
-		(property "Description" "part selected: TS-1187A-B-A-B"
+		(property "Description" "part selected: TC-1109-C-E"
 			(at 205.74 246.38 0)
 			(hide yes)
@@
 			)
 		)
-		(property "Footprint" "Button_Switch_SMD:SW_Push_1P1T_XKB_TS-1187A"
+		(property "Footprint" "XKB Connection:TC-1109-C-E"
 			(at 449.58 241.3 0)
 			(hide yes)
@@
 			)
 		)
-		(property "Description" "part selected: TS-1187A-B-A-B"
+		(property "Description" "part selected: TC-1109-C-E"
 			(at 449.58 246.38 0)
 			(hide yes)

Commit message: feat(v1 hardware): new starter pcb
Parts:
- SW73, SW74, SW75, SW76, SW77, SW82, SW83, SW84, SW85, SW86: footprint Amazon:1208YD -> ALPS Electric:SSSS820201
- SW78, SW79, SW80, SW81: footprint Amazon:1208YD -> ALPS Electric:SPEF110100
Changed lines of the file:
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@@
 		(title "Slack")
 		(date "2026-07-25")
-		(rev "A.0.4")
+		(rev "A.0.5")
 	)
 	(text "Latch Row"
@@
 			)
 		)
-		(property "Footprint" "Amazon:1208YD"
+		(property "Footprint" "ALPS Electric:SSSS820201"
 			(at 124.46 304.8 0)
 			(hide yes)
@@
 			)
 		)
-		(property "Footprint" "Amazon:1208YD"
+		(property "Footprint" "ALPS Electric:SSSS820201"
 			(at 533.4 304.8 0)
 			(hide yes)
@@
 			)
 		)
-		(property "Footprint" "Amazon:1208YD"
+		(property "Footprint" "ALPS Electric:SSSS820201"
 			(at 96.52 304.8 0)
 			(hide yes)
@@
 			)
 		)
-		(property "Footprint" "Amazon:1208YD"
+		(property "Footprint" "ALPS Electric:SSSS820201"
 			(at 505.46 304.8 0)
 			(hide yes)
@@
 			)
 		)
-		(property "Footprint" "Amazon:1208YD"
+		(property "Footprint" "ALPS Electric:SSSS820201"
 			(at 40.64 304.8 0)
 			(hide yes)
@@
 			)
 		)
-		(property "Footprint" "Amazon:1208YD"
+		(property "Footprint" "ALPS Electric:SSSS820201"
 			(at 617.22 304.8 0)
 			(hide yes)
@@
 			)
 		)
-		(property "Footprint" "Amazon:1208YD"
+		(property "Footprint" "ALPS Electric:SPEF110100"
 			(at 208.28 304.8 0)
 			(hide yes)
@@
 			)
 		)
-		(property "Footprint" "Amazon:1208YD"
+		(property "Footprint" "ALPS Electric:SPEF110100"
 			(at 180.34 304.8 0)
 			(hide yes)
@@
 			)
 		)
-		(property "Footprint" "Amazon:1208YD"
+		(property "Footprint" "ALPS Electric:SSSS820201"
 			(at 561.34 304.8 0)
 			(hide yes)
@@
 			)
 		)
-		(property "Footprint" "Amazon:1208YD"
+		(property "Footprint" "ALPS Electric:SSSS820201"
 			(at 68.58 304.8 0)
 			(hide yes)
@@
 			)
 		)
-		(property "Footprint" "Amazon:1208YD"
+		(property "Footprint" "ALPS Electric:SPEF110100"
 			(at 477.52 304.8 0)
 			(hide yes)
@@
 			)
 		)
-		(property "Footprint" "Amazon:1208YD"
+		(property "Footprint" "ALPS Electric:SSSS820201"
 			(at 589.28 304.8 0)
 			(hide yes)
@@
 			)
 		)
-		(property "Footprint" "Amazon:1208YD"
+		(property "Footprint" "ALPS Electric:SPEF110100"
 			(at 452.12 304.8 0)
 			(hide yes)
@@
 			)
 		)
-		(property "Footprint" "Amazon:1208YD"
+		(property "Footprint" "ALPS Electric:SSSS820201"
 			(at 152.4 304.8 0)
 			(hide yes)

Commit message: feat(v1 hardware): added schematic symbols for latches
Parts:
- SW73, SW74, SW75, SW76, SW77, SW82, SW83, SW84, SW85, SW86: value SW_DIP_x01 -> SSSS820201; symbol Switch:SW_DIP_x01 -> ALPS Electric:SSSS820201
- SW78, SW79, SW80, SW81: value SW_DIP_x01 -> SPEF110100; footprint ALPS Electric:SPEF110100 -> SPEF110100; symbol Switch:SW_DIP_x01 -> ALPS Electric:SPEF110100; Arrow Part Number (none) -> SPEF110100; Arrow Price/Stock (none) -> https://www.arrow.com/en/products/spef110100/alpsalpine.htm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; Height (none) -> 14.6; Manufacturer_Name (none) -> ALPS Electric; Manufacturer_Part_Number (none) -> SPEF110100; Mouser Part Number (none) -> 688-SPEF110100; Mouser Price/Stock (none) -> https://www.mouser.co.uk/ProductDetail/Alps-Alpine/SPEF1101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
Connections:
- net Column1: now also SW73.2 (C); no longer SW73.1
- net Column10: now also SW82.2 (C); no longer SW82.1
- net Column11: now also SW83.2 (C); no longer SW83.1
- net Column12: now also SW84.2 (C); no longer SW84.1
- net Column13: now also SW85.2 (C); no longer SW85.1
- net Column14: now also SW86.2 (C); no longer SW86.1
- net Column2: now also SW74.2 (C); no longer SW74.1
- net Column3: now also SW75.2 (C); no longer SW75.1
- net Column4: now also SW76.2 (C); no longer SW76.1
- net Column5: now also SW77.2 (C); no longer SW77.1
- net Column6: now also SW78.C1 (C), SW78.C2 (C); no longer SW78.1
- net Column7: now also SW79.C1 (C), SW79.C2 (C); no longer SW79.1
- net Column8: now also SW80.C1 (C), SW80.C2 (C); no longer SW80.1
- net Column9: now also SW81.C1 (C), SW81.C2 (C); no longer SW81.1
- net at D74.2 (A): now also SW74.4; no longer SW74.2
- net at D76.2 (A): now also SW76.4; no longer SW76.2
- net at D85.2 (A): now also SW85.4; no longer SW85.2
- net at D83.2 (A): now also SW83.4; no longer SW83.2
- net at D75.2 (A): now also SW75.4; no longer SW75.2
- net at D82.2 (A): now also SW82.4; no longer SW82.2
- net at D73.2 (A): now also SW73.4; no longer SW73.2
- net at D86.2 (A): now also SW86.4; no longer SW86.2
- net at D84.2 (A): now also SW84.4; no longer SW84.2
- net at D77.2 (A): now also SW77.4; no longer SW77.2
- new net GND: SW73.7 (H), SW74.7 (H), SW75.7 (H), SW76.7 (H), SW77.7 (H), SW78.MH1 (MH), SW78.MH2 (MH), SW78.MH3 (MH), SW78.MH4 (MH), SW79.MH1 (MH), SW79.MH2 (MH), SW79.MH3 (MH), SW79.MH4 (MH), SW80.MH1 (MH), SW80.MH2 (MH), SW80.MH3 (MH), SW80.MH4 (MH), SW81.MH1 (MH), SW81.MH2 (MH), SW81.MH3 (MH), SW81.MH4 (MH), SW82.7 (H), SW83.7 (H), SW84.7 (H), SW85.7 (H), SW86.7 (H)
- no-connect marks 0 -> 44

Commit message: feat(v1 hardware): aligned schematic symbols with pcb footprints
Parts:
- RE1/SW7, RE2/SW8, RE3/SW21, RE4/SW22, RE5/SW35, RE6/SW36, RE7/SW49, RE8/SW50: value RotaryEncoder_Switch -> PEC11S-929K-S0015; symbol Device:RotaryEncoder_Switch -> Bourns:PEC11S-929K-S0015; Arrow Part Number (none) -> PEC11S-929K-S0015; Arrow Price/Stock (none) -> https://www.arrow.com/en/products/pec11s-929k-s0015/bourns?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; Height (none) -> 14; Manufacturer_Name (none) -> Bourns; Manufacturer_Part_Number (none) -> PEC11S-929K-S0015; Mouser Part Number (none) -> 652-PEC11S929K-S0015; Mouser Price/Stock (none) -> https://www.mouser.co.uk/ProductDetail/Bourns/PEC11S-929K-S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
- RE10, RE9: value RotaryEncoder -> EC10E1220505; symbol Device:RotaryEncoder -> ALPS Electric:EC10E1220505; Height (none) -> 10.6; Manufacturer_Name (none) -> ALPS Electric; Manufacturer_Part_Number (none) -> EC10E1220505; Mouser Part Number (none) -> 688-EC10E1220505; Mouser Price/Stock (none) -> https://www.mouser.co.uk/ProductDetail/Alps-Alpine/EC10E122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
- SW1, SW10, SW11, SW12, SW13, SW14, SW15, SW16, SW17, SW18, SW19, SW2, SW20, SW23, SW24, SW25, SW26, SW27, SW28, SW29, SW3, SW30, SW31, SW32, SW33, SW34, SW37, SW38, SW39, SW4, SW40, SW41, SW42, SW43, SW44, SW45, SW46, SW47, SW48, SW5, SW51, SW52, SW53, SW54, SW55, SW56, SW57, SW58, SW59, SW6, SW60, SW61, SW62, SW67, SW68, SW69, SW70, SW71, SW72, SW9: symbol Switch:SW_Push_45deg -> Cherry:MX6C-K3NB
- SW78, SW79, SW80, SW81: footprint SPEF110100 -> ALPS Electric:SPEF110100
Connections:
- net GND is gone; now on net DGND: SW73.7 (H), SW74.7 (H), SW75.7 (H), SW76.7 (H), SW77.7 (H), SW78.MH1 (MH), SW78.MH2 (MH), SW78.MH3 (MH), SW78.MH4 (MH), SW79.MH1 (MH), SW79.MH2 (MH), SW79.MH3 (MH), SW79.MH4 (MH), SW80.MH1 (MH), SW80.MH2 (MH), SW80.MH3 (MH), SW80.MH4 (MH), SW81.MH1 (MH), SW81.MH2 (MH), SW81.MH3 (MH), SW81.MH4 (MH), SW82.7 (H), SW83.7 (H), SW84.7 (H), SW85.7 (H), SW86.7 (H)
- net Column7: now also RE1/SW7.D1 (SI), RE3/SW21.D1 (SI), RE5/SW35.D1 (SI), RE7/SW49.D1 (SI); no longer RE1/SW7.S2, RE3/SW21.S2, RE5/SW35.S2, RE7/SW49.S2
- net Column8: now also RE2/SW8.D1 (SI), RE4/SW22.D1 (SI), RE6/SW36.D1 (SI), RE8/SW50.D1 (SI); no longer RE2/SW8.S1, RE4/SW22.S1, RE6/SW36.S1, RE8/SW50.S1
- net DGND: now also RE1/SW7.C1 (C), RE1/SW7.MP1 (H), RE1/SW7.MP2 (H), RE1/SW7.MP3 (H), RE1/SW7.MP4 (H), RE1/SW7.MP5 (H), RE1/SW7.MP6 (H), RE10.C1 (C), RE10.MH1 (H), RE10.MH2 (H), RE2/SW8.C1 (C), RE2/SW8.MP1 (H), RE2/SW8.MP2 (H), RE2/SW8.MP3 (H), RE2/SW8.MP4 (H), RE2/SW8.MP5 (H), RE2/SW8.MP6 (H), RE3/SW21.C1 (C), RE3/SW21.MP1 (H), RE3/SW21.MP2 (H), RE3/SW21.MP3 (H), RE3/SW21.MP4 (H), RE3/SW21.MP5 (H), RE3/SW21.MP6 (H), RE4/SW22.C1 (C), RE4/SW22.MP1 (H), RE4/SW22.MP2 (H), RE4/SW22.MP3 (H), RE4/SW22.MP4 (H), RE4/SW22.MP5 (H), RE4/SW22.MP6 (H), RE5/SW35.C1 (C), RE5/SW35.MP1 (H), RE5/SW35.MP2 (H), RE5/SW35.MP3 (H), RE5/SW35.MP4 (H), RE5/SW35.MP5 (H), RE5/SW35.MP6 (H), RE6/SW36.C1 (C), RE6/SW36.MP1 (H), RE6/SW36.MP2 (H), RE6/SW36.MP3 (H), RE6/SW36.MP4 (H), RE6/SW36.MP5 (H), RE6/SW36.MP6 (H), RE7/SW49.C1 (C), RE7/SW49.MP1 (H), RE7/SW49.MP2 (H), RE7/SW49.MP3 (H), RE7/SW49.MP4 (H), RE7/SW49.MP5 (H), RE7/SW49.MP6 (H), RE8/SW50.C1 (C), RE8/SW50.MP1 (H), RE8/SW50.MP2 (H), RE8/SW50.MP3 (H), RE8/SW50.MP4 (H), RE8/SW50.MP5 (H), RE8/SW50.MP6 (H), RE9.C1 (C), RE9.MH1 (H), RE9.MH2 (H); no longer RE1/SW7.C, RE10.C, RE2/SW8.C, RE3/SW21.C, RE4/SW22.C, RE5/SW35.C, RE6/SW36.C, RE7/SW49.C, RE8/SW50.C, RE9.C
- net RotaryEncoder_AChannel1: now also C1.1, R2.1; no longer C2.1, R4.1
- net RotaryEncoder_AChannel3: now also C5.1, R10.2; no longer C6.1, R12.1
- net RotaryEncoder_AChannel5: now also C9.1, R18.1; no longer C10.1, R20.1
- net RotaryEncoder_AChannel7: now also C13.1, R27.1; no longer C14.1, R28.1
- net RotaryEncoder_AChannel9: now also C17.1, R34.1; no longer C18.1, R36.1
- net RotaryEncoder_BChannel1: now also C2.1, R4.1; no longer C1.1, R2.1
- net RotaryEncoder_BChannel3: now also C6.1, R12.1; no longer C5.1, R10.2
- net RotaryEncoder_BChannel5: now also C10.1, R20.1; no longer C9.1, R18.1
- net RotaryEncoder_BChannel7: now also C14.1, R28.1; no longer C13.1, R27.1
- net RotaryEncoder_BChannel9: now also C18.1, R36.1; no longer C17.1, R34.1
- net at R25.2, R27.2: now also RE7/SW49.A1 (A); no longer RE7/SW49.B
- net at R15.1, R16.2: now also RE4/SW22.B1 (B); no longer RE4/SW22.B
- net at R10.1, R9.2: now also RE3/SW21.A1 (A); no longer RE3/SW21.B
- net at D22.2 (A): now also RE4/SW22.E1 (SO); no longer RE4/SW22.S2
- net at R29.2, R30.2: now also RE8/SW50.A1 (A); no longer RE8/SW50.A
- net at R35.2, R4.2: now also RE1/SW7.B1 (B); no longer RE1/SW7.A
- net at R17.2, R18.2: now also RE5/SW35.A1 (A); no longer RE5/SW35.B
- net at R13.2, R14.1: now also RE4/SW22.A1 (A); no longer RE4/SW22.A
- net at R33.2, R34.2: now also RE9.A1 (A); no longer RE9.B
- net at R3.2, R36.2: now also RE9.B1 (B); no longer RE9.A
- net at R19.1, R20.2: now also RE5/SW35.B1 (B); no longer RE5/SW35.A
- net at R11.2, R28.2: now also RE7/SW49.B1 (B); no longer RE7/SW49.A
- net at D35.2 (A): now also RE5/SW35.E1 (SO); no longer RE5/SW35.S1
- net at R31.2, R32.2: now also RE8/SW50.B1 (B); no longer RE8/SW50.B
- net at D8.2 (A): now also RE2/SW8.E1 (SO); no longer RE2/SW8.S2
- net at R5.2, R6.2: now also RE2/SW8.A1 (A); no longer RE2/SW8.A
- net at R7.2, R8.2: now also RE2/SW8.B1 (B); no longer RE2/SW8.B
- net at R21.1, R22.2: now also RE6/SW36.A1 (A); no longer RE6/SW36.A
- net at R12.2, R26.1: now also RE3/SW21.B1 (B); no longer RE3/SW21.A
- net at D49.2 (A): now also RE7/SW49.E1 (SO); no longer RE7/SW49.S1
- net at R1.2, R2.2: now also RE1/SW7.A1 (A); no longer RE1/SW7.B
- net at R23.1, R24.1: now also RE6/SW36.B1 (B); no longer RE6/SW36.B
- net at D7.2 (A): now also RE1/SW7.E1 (SO); no longer RE1/SW7.S1
- net at R39.2, R40.1: now also RE10.B1 (B); no longer RE10.B
- net at D36.2 (A): now also RE6/SW36.E1 (SO); no longer RE6/SW36.S2
- net at D50.2 (A): now also RE8/SW50.E1 (SO); no longer RE8/SW50.S2
- net at D21.2 (A): now also RE3/SW21.E1 (SO); no longer RE3/SW21.S1
- net at R37.2, R38.2: now also RE10.A1 (A); no longer RE10.A

Commit message: feat(v1 hardware): transfer to ergogen layout
Parts:
- removed D57, D72: D, Diode_SMD:D_SOD-523, symbol Device:D
- removed SW57, SW72: MSwitch, Cherry:Cherry_ULP_SMD, symbol Cherry:MX6C-K3NB
- renumbered D58 to D57, D59 to D58, D60 to D59, D61 to D60, D62 to D61, D63 to D62, D66 to D63, D67 to D64, D68 to D65, D69 to D66, D70 to D67, D71 to D68, D73 to D69, D74 to D70, D75 to D71, D76 to D72, D77 to D73, D78 to D74, D79 to D75, D80 to D76, D81 to D77, D82 to D78, D83 to D79, D84 to D80, D85 to D81, D86 to D82, SW58 to SW57, SW59 to SW58, SW60 to SW59, SW61 to SW60, SW62 to SW61, SW63 to SW62, SW66 to SW63, SW67 to SW64, SW68 to SW65, SW69 to SW66, SW70 to SW67, SW71 to SW68, SW73 to SW69, SW74 to SW70, SW75 to SW71, SW76 to SW72, SW77 to SW73, SW78 to SW74, SW79 to SW75, SW80 to SW76, SW81 to SW77, SW82 to SW78, SW83 to SW79, SW84 to SW80, SW85 to SW81, SW86 to SW82

Commit message: feat(v1 hardware): mid component update save
Parts:
- SW62: footprint XKB Connection:TC-1109-C-E -> ALPS Electric:SKQGAKE010
Changed lines of the file:
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@@
 			)
 		)
-		(property "Footprint" "XKB Connection:TC-1109-C-E"
+		(property "Footprint" "ALPS Electric:SKQGAKE010"
 			(at 205.74 241.3 0)
 			(hide yes)
@@
 			)
 		)
-		(property "Description" "part selected: TC-1109-C-E"
+		(property "Description" "part selected: SKQGAKE010"
 			(at 205.74 246.38 0)
 			(hide yes)
@@
 			)
 		)
-		(property "Description" "part selected: TC-1109-C-E"
+		(property "Description" "part selected: TC-1109"
 			(at 449.58 246.38 0)
 			(hide yes)

Commit message: feat(v1 hardware): review fixes
Parts:
- D1, D10, D11, D12, D13, D14, D15, D16, D17, D18, D19, D2, D20, D21, D22, D23, D24, D25, D26, D27, D28, D29, D3, D30, D31, D32, D33, D34, D35, D36, D37, D38, D39, D4, D40, D41, D42, D43, D44, D45, D46, D47, D48, D49, D5, D50, D51, D52, D53, D54, D55, D56, D57, D58, D59, D6, D60, D61, D62, D63, D64, D65, D66, D67, D68, D69, D7, D70, D71, D72, D73, D74, D75, D76, D77, D78, D79, D8, D80, D81, D82, D9: value D -> BAS16TS
