File: hardware/v1-electronics/slack.kicad_pcb (KiCad board)
At the start: 2 copper layers, 399.2 x 265.1 mm, 410 parts, among them IC1 TPS61288LRQQR, IC2 MP2721GRH-0000-Z, IC3 IS31FL3733-QFLS4-TR, IC4 IS31FL3733-QFLS4-TR, J1 Female USB-C USB2.0, J2 XT30PW-M, J3 Female JST-SH, Q1 AON7423, SW1 MSwitch, SW10 MSwitch, SW11 MSwitch, SW12 MSwitch, SW13 MSwitch, SW14 MSwitch, SW15 MSwitch, SW16 MSwitch, SW17 MSwitch, SW18 MSwitch, SW19 MSwitch, SW2 MSwitch, SW20 MSwitch, SW23 MSwitch, SW24 MSwitch, SW25 MSwitch, SW26 MSwitch, SW27 MSwitch, SW28 MSwitch, SW29 MSwitch, SW3 MSwitch, SW30 MSwitch, SW31 MSwitch, SW32 MSwitch, SW33 MSwitch, SW34 MSwitch, SW37 MSwitch, SW38 MSwitch, SW39 MSwitch, SW4 MSwitch, SW40 MSwitch, SW41 MSwitch, SW42 MSwitch, SW43 MSwitch, SW44 MSwitch, SW45 MSwitch, SW46 MSwitch, SW47 MSwitch, SW48 MSwitch, SW5 MSwitch, SW51 MSwitch, SW52 MSwitch, SW53 MSwitch, SW54 MSwitch, SW55 MSwitch, SW56 MSwitch, SW57 MSwitch, SW58 MSwitch, SW59 MSwitch, SW6 MSwitch, SW60 MSwitch, SW61 MSwitch, SW62 SW_Push, SW63 SW_Push, SW64 MSwitch, SW65 MSwitch, SW66 MSwitch, SW67 MSwitch, SW68 MSwitch, SW69 SSSS820201, SW7 2TED3M6RES, SW70 SSSS820201, SW71 SSSS820201, SW72 SSSS820201, SW73 SSSS820201, SW74 SPEF110100, SW75 SPEF110100, SW76 SPEF110100, SW77 SPEF110100, SW78 SSSS820201, SW79 SSSS820201, SW8 SW_Push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

Commit message: feat(v1 hardware): place mounting holes
Parts:
- added H1: MountingHole_2.2mm_M2_Pad_Via, MountingHole_2.2mm_M2_Pad_Via, F.Cu at (147.2, 52.8)
- added H10: MountingHole_2.2mm_M2_Pad_Via, MountingHole_2.2mm_M2_Pad_Via, F.Cu at (347.1, 162.6)
- added H11: MountingHole_2.2mm_M2_Pad_Via, MountingHole_2.2mm_M2_Pad_Via, F.Cu at (140.3, 201.2)
- added H12: MountingHole_2.2mm_M2_Pad_Via, MountingHole_2.2mm_M2_Pad_Via, F.Cu at (302.6, 201.2)
- added H13: MountingHole_2.2mm_M2_Pad_Via, MountingHole_2.2mm_M2_Pad_Via, F.Cu at (221.4, 132.1)
- added H14: MountingHole_2.2mm_M2_Pad_Via, MountingHole_2.2mm_M2_Pad_Via, F.Cu at (221.4, 196.3)
- added H2: MountingHole_2.2mm_M2_Pad_Via, MountingHole_2.2mm_M2_Pad_Via, F.Cu at (295.7, 52.8)
- added H3: MountingHole_2.2mm_M2_Pad_Via, MountingHole_2.2mm_M2_Pad_Via, F.Cu at (71.8, 70.7)
- added H4: MountingHole_2.2mm_M2_Pad_Via, MountingHole_2.2mm_M2_Pad_Via, F.Cu at (371.1, 70.7)
- added H5: MountingHole_2.2mm_M2_Pad_Via, MountingHole_2.2mm_M2_Pad_Via, F.Cu at (57.1, 153.5)
- added H6: MountingHole_2.2mm_M2_Pad_Via, MountingHole_2.2mm_M2_Pad_Via, F.Cu at (385.7, 153.5)
- added H7: MountingHole_2.2mm_M2_Pad_Via, MountingHole_2.2mm_M2_Pad_Via, F.Cu at (166.8, 169.2)
- added H8: MountingHole_2.2mm_M2_Pad_Via, MountingHole_2.2mm_M2_Pad_Via, F.Cu at (276.1, 169.2)
- added H9: MountingHole_2.2mm_M2_Pad_Via, MountingHole_2.2mm_M2_Pad_Via, F.Cu at (95.8, 162.6)
- moved U1 165.0 mm to (221.1, 83.0), turned to 0 degrees
- moved C1 20.3 mm to (140.1, 263.2)
- moved C10 20.3 mm to (143.0, 271.1)
- moved C11 20.3 mm to (145.9, 263.2)
- moved C13 20.3 mm to (145.9, 267.2)
- moved C15 20.3 mm to (145.9, 271.1)
- moved C16 20.3 mm to (148.8, 263.2)
- moved C18 20.3 mm to (148.8, 267.2)
- moved C20 20.3 mm to (148.8, 271.1)
- moved C3 20.3 mm to (140.1, 267.2)
- moved C5 20.3 mm to (140.1, 271.1)
- moved C51 20.3 mm to (225.6, 261.8)
- moved C52 20.3 mm to (225.6, 264.8)
- moved C6 20.3 mm to (143.0, 263.2)
- moved C8 20.3 mm to (143.0, 267.2)
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Other:
- board size 399.2 x 265.1 mm -> 335.2 x 170.7 mm

Commit message: feat(v1 hardware): set base pcb outline
Other:
- board size 335.2 x 170.7 mm -> 339 x 170.5 mm

Commit message: feat(v1 hardware): update config switch
Parts:
- C21, C22, C23, C24, C25, C26, C27, C28, C29, C30, C31, C32, C33, C34, C35, C36, IC3, IC4, J1, J2, LED511, LED512, LED513, LED514, LED515, LED517, LED518, LED521, LED522, LED523, LED524, LED525, LED526, LED527, R41, R42, R43, R45, R46, R47, SW7, TH1, U1: moved to B.Cu
- JP1: footprint Connector_PinHeader_2.54mm:PinHeader_1x02_P2.54mm_Vertical -> Dongguan Guangzhu Industrial:DSIC01LSGET; moved to B.Cu
- JP2, JP3, JP4, JP5, JP6: footprint Connector_PinHeader_2.54mm:PinHeader_1x02_P2.54mm_Vertical -> Dongguan Guangzhu Industrial:DSIC01LSGET
- moved J1 145.8 mm to (72.9, 88.2), turned to 80 degrees
- moved TH1 127.6 mm to (115.9, 61.9), turned to -10 degrees
- moved J2 115.2 mm to (109.5, 62.1), turned to -10 degrees
- moved SW7 79.1 mm to (172.5, 78.3), turned to 170 degrees
- moved LED527 77.6 mm to (420.0, 145.9)
- moved LED518 69.9 mm to (23.7, 152.7)
- moved R47 69.8 mm to (404.3, 149.8)
- moved R43 69.7 mm to (36.4, 152.8)
- moved LED526 69.2 mm to (420.0, 150.2)
- moved R45 69.0 mm to (407.8, 150.2)
- moved R41 68.9 mm to (39.8, 153.2)
- moved C33 65.6 mm to (399.9, 152.0)
- moved C36 65.4 mm to (32.0, 155.0)
- moved C26 64.3 mm to (409.4, 152.7)
- moved R46 64.1 mm to (404.3, 152.8)
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Connections:
- SW62 pad 3: /MCU/Column7 -> (no net)
- SW62 pad 4: Net-(D62-A) -> (no net)
Other:
- copper layers 2 -> 4
