File: hardware/v1-electronics/slack.kicad_pcb (KiCad board)
At the start: 4 copper layers, 339 x 170.5 mm, 424 parts, among them IC1 TPS61288LRQQR, IC2 MP2721GRH-0000-Z, IC3 IS31FL3733-QFLS4-TR, IC4 IS31FL3733-QFLS4-TR, J1 Female USB-C USB2.0, J2 XT30PW-M, J3 Female JST-SH, Q1 AON7423, SW1 MSwitch, SW10 MSwitch, SW11 MSwitch, SW12 MSwitch, SW13 MSwitch, SW14 MSwitch, SW15 MSwitch, SW16 MSwitch, SW17 MSwitch, SW18 MSwitch, SW19 MSwitch, SW2 MSwitch, SW20 MSwitch, SW23 MSwitch, SW24 MSwitch, SW25 MSwitch, SW26 MSwitch, SW27 MSwitch, SW28 MSwitch, SW29 MSwitch, SW3 MSwitch, SW30 MSwitch, SW31 MSwitch, SW32 MSwitch, SW33 MSwitch, SW34 MSwitch, SW37 MSwitch, SW38 MSwitch, SW39 MSwitch, SW4 MSwitch, SW40 MSwitch, SW41 MSwitch, SW42 MSwitch, SW43 MSwitch, SW44 MSwitch, SW45 MSwitch, SW46 MSwitch, SW47 MSwitch, SW48 MSwitch, SW5 MSwitch, SW51 MSwitch, SW52 MSwitch, SW53 MSwitch, SW54 MSwitch, SW55 MSwitch, SW56 MSwitch, SW57 MSwitch, SW58 MSwitch, SW59 MSwitch, SW6 MSwitch, SW60 MSwitch, SW61 MSwitch, SW62 SW_Push, SW63 SW_Push, SW64 MSwitch, SW65 MSwitch, SW66 MSwitch, SW67 MSwitch, SW68 MSwitch, SW69 SSSS820201, SW7 2TED3M6RES, SW70 SSSS820201, SW71 SSSS820201, SW72 SSSS820201, SW73 SSSS820201, SW74 SPEF110100, SW75 SPEF110100, SW76 SPEF110100, SW77 SPEF110100, SW78 SSSS820201, SW79 SSSS820201, SW8 SW_Push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

Commit message: feat(v1 hardware):update outline
Parts:
- moved J1 2.71 mm to (70.2, 87.7)
Other:
- board size 339 x 170.5 mm -> 338.9 x 170.5 mm
Changed lines of the file:
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@@
 	(footprint "Connector_USB:USB_C_Receptacle_GCT_USB4085"
 		(layer "B.Cu")
-		(at 72.883884 88.196945 80)
+		(at 70.2168 87.7268 80)
 		(descr "USB 2.0 Type C Receptacle, https://gct.co/Files/Drawings/USB4085.pdf")
 		(tags "USB Type-C Receptacle Through-hole Right angle")
@@
 		(pts
 			(arc
-				(start 248.93 74.2937)
-				(mid 250.3997 73.4905)
-				(end 250.7292 71.7827)
+				(start 241.0678 74.2937)
+				(mid 241.8195 74.1471)
+				(end 242.461 73.7287)
 			)
 			(arc
-				(start 249.8974 67.7977)
-				(mid 250.2698 66.335)
-				(end 251.6382 65.5348)
-			)
-			(arc
-				(start 267.9807 62.657)
-				(mid 268.2237 62.6392)
-				(end 268.8022 62.5435)
+				(start 250.2973 66.1209)
+				(mid 250.7819 65.7741)
+				(end 251.3471 65.5855)
 			)
+			(xy 268.8022 62.5435)
 			(arc
 				(start 279.7043 60.5875)
@@
 			)
 			(arc
-				(start 390.9207 156.0679)
-				(mid 390.4797 157.5455)
-				(end 389.0378 158.2791)
+				(start 390.8646 155.7494)
+				(mid 390.5332 157.2438)
+				(end 389.2422 158.0663)
 			)
 			(arc
-				(start 351.924 162.2776)
-				(mid 351.1607 162.5836)
-				(end 350.5425 163.2283)
+				(start 350.0361 164.9794)
+				(mid 349.3078 165.2628)
+				(end 348.7437 165.8038)
 			)
 			(arc
@@
 			)
 			(arc
-				(start 92.3543 163.2283)
-				(mid 91.7361 162.5836)
-				(end 90.9728 162.2776)
+				(start 94.1531 165.8038)
+				(mid 93.589 165.2628)
+				(end 92.8607 164.9794)
 			)
 			(arc
-				(start 53.859 158.2791)
-				(mid 52.4171 157.5455)
-				(end 51.9761 156.0679)
+				(start 53.6546 158.0663)
+				(mid 52.3636 157.2438)
+				(end 52.0322 155.7494)
 			)
 			(arc
@@
 				(end 163.1925 60.5875)
 			)
+			(xy 174.0946 62.5435)
 			(arc
-				(start 174.0946 62.5435)
-				(mid 174.6731 62.6392)
-				(end 174.9161 62.657)
-			)
-			(arc
-				(start 191.2586 65.5348)
-				(mid 192.627 66.335)
-				(end 192.9994 67.7977)
+				(start 191.5497 65.5855)
+				(mid 192.1149 65.7741)
+				(end 192.5995 66.1209)
 			)
 			(arc
-				(start 192.1676 71.7827)
-				(mid 192.4971 73.4905)
-				(end 193.9668 74.2937)
+				(start 200.4358 73.7287)
+				(mid 201.0773 74.1471)
+				(end 201.829 74.2937)
 			)
 		)
@@
 		)
 		(fill no)
-		(locked yes)
 		(layer "Edge.Cuts")
 	)
 	(gr_line
-		(start 48.045 152.785)
-		(end 93.715 161.075)
-		(stroke
-			(width 1)
-			(type default)
-		)
-		(layer "User.3")
-	)
-	(gr_line
 		(start 53.165 149.015)
 		(end 66.535 74.145)
@@
 			(type default)
 		)
-		(layer "User.3")
-	)
-	(gr_line
-		(start 201.22 74.49)
-		(end 192.475 66)
-		(stroke
-			(width 1)
-			(type default)
-		)

Commit message: feat(v1 hardware): add 3D model for config switches
Connections:
- J1 pad A1: Net-(J1-GND-PadA1) -> DGND
- J1 pad A12: Net-(J1-GND-PadA1) -> DGND
- J1 pad B1: Net-(J1-GND-PadA1) -> DGND
- J1 pad B12: Net-(J1-GND-PadA1) -> DGND
- J1 pad SH: unconnected-(J1-SHIELD-PadSH) -> DGND
Changed lines of the file:
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@@
 		(sheetname "/MCU/")
 		(sheetfile "controller.kicad_sch")
-		(units
-			(unit
-				(name "A")
-				(pins "1" "2")
-			)
-		)
 		(attr smd)
 		(duplicate_pad_numbers_are_jumpers no)
@@
 		)
 		(embedded_fonts no)
+		(model "${KIPRJMOD}/Dongguan Guangzhu Industrial/DSIC01LSGET.step"
+			(offset
+				(xyz 0 0 0)
+			)
+			(scale
+				(xyz 1 1 1)
+			)
+			(rotate
+				(xyz 0 0 0)
+			)
+		)
 	)
 	(footprint "Resistor_SMD:R_0805_2012Metric"
@@
 		(sheetname "/MCU/")
 		(sheetfile "controller.kicad_sch")
-		(units
-			(unit
-				(name "A")
-				(pins "1" "2")
-			)
-		)
 		(attr smd)
 		(duplicate_pad_numbers_are_jumpers no)
@@
 		)
 		(embedded_fonts no)
+		(model "${KIPRJMOD}/Dongguan Guangzhu Industrial/DSIC01LSGET.step"
+			(offset
+				(xyz 0 0 0)
+			)
+			(scale
+				(xyz 1 1 1)
+			)
+			(rotate
+				(xyz 0 0 0)
+			)
+		)
 	)
 	(footprint "Bourns:PEC11S929KS0015"
@@
 		(sheetname "/Power Train/")
 		(sheetfile "power.kicad_sch")
-		(units
-			(unit
-				(name "A")
-				(pins "1" "2")
-			)
-		)
 		(attr smd)
 		(duplicate_pad_numbers_are_jumpers no)
@@
 		)
 		(embedded_fonts no)
+		(model "${KIPRJMOD}/Dongguan Guangzhu Industrial/DSIC01LSGET.step"
+			(offset
+				(xyz 0 0 0)
+			)
+			(scale
+				(xyz 1 1 1)
+			)
+			(rotate
+				(xyz 0 0 0)
+			)
+		)
 	)
 	(footprint "Resistor_SMD:R_0805_2012Metric"
@@
 		(sheetname "/MCU/")
 		(sheetfile "controller.kicad_sch")
-		(units
-			(unit
-				(name "A")
-				(pins "1" "2")
-			)
-		)
 		(attr smd)
 		(duplicate_pad_numbers_are_jumpers no)
@@
 		)
 		(embedded_fonts no)
+		(model "${KIPRJMOD}/Dongguan Guangzhu Industrial/DSIC01LSGET.step"
+			(offset
+				(xyz 0 0 0)
+			)
+			(scale
+				(xyz 1 1 1)
+			)
+			(rotate
+				(xyz 0 0 0)
+			)
+		)
 	)
 	(footprint "MountingHole_2.2mm_M2_Pad_Via"
@@
 		(sheetname "/Power Train/")
 		(sheetfile "power.kicad_sch")
-		(units
-			(unit
-				(name "A")
-				(pins "1" "2")
-			)
-		)
 		(attr smd)
 		(duplicate_pad_numbers_are_jumpers no)
@@
 		)
 		(embedded_fonts no)
+		(model "${KIPRJMOD}/Dongguan Guangzhu Industrial/DSIC01LSGET.step"
+			(offset
+				(xyz 0 0 0)
+			)
+			(scale
+				(xyz 1 1 1)
+			)
+			(rotate
+				(xyz 0 0 0)
+			)
+		)
 	)
 	(footprint "Capacitor_SMD:C_0805_2012Metric"
@@
 		(sheetname "/LED Matricies/")
 		(sheetfile "led_matrix.kicad_sch")
-		(units
-			(unit
-				(name "A")
-				(pins "1" "2")
-			)
-		)
 		(attr smd)
 		(duplicate_pad_numbers_are_jumpers no)
@@
 		)
 		(embedded_fonts no)
+		(model "${KIPRJMOD}/Dongguan Guangzhu Industrial/DSIC01LSGET.step"
+			(offset
+				(xyz 0 0 0)
+			)
+			(scale
+				(xyz 1 1 1)
+			)
+			(rotate
+				(xyz 0 0 0)
+			)
+		)
 	)
 	(footprint "Capacitor_Tantalum_SMD:CP_EIA-3216-18_Kemet-A"
@@
 			(layers "*.Cu" "*.Mask")
 			(remove_unused_layers no)
-			(net "Net-(J1-GND-PadA1)")
+			(net "DGND")
 			(pinfunction "GND_A1")
 			(pintype "passive")
@@
 			(layers "*.Cu" "*.Mask")
 			(remove_unused_layers no)
-			(net "Net-(J1-GND-PadA1)")
+			(net "DGND")
 			(pinfunction "GND_A12")
 			(pintype "passive")
@@
 			(layers "*.Cu" "*.Mask")
 			(remove_unused_layers no)
-			(net "Net-(J1-GND-PadA1)")
+			(net "DGND")
 			(pinfunction "GND_B1")
 			(pintype "passive")
@@
 			(layers "*.Cu" "*.Mask")
 			(remove_unused_layers no)
-			(net "Net-(J1-GND-PadA1)")
+			(net "DGND")
 			(pinfunction "GND_B12")
 			(pintype "passive")
@@
 			(layers "*.Cu" "*.Mask")
 			(remove_unused_layers no)
-			(net "unconnected-(J1-SHIELD-PadSH)")
+			(net "DGND")
 			(pinfunction "SHIELD_SH")
 			(pintype "passive")
@@
 			(layers "*.Cu" "*.Mask")
 			(remove_unused_layers no)
-			(net "unconnected-(J1-SHIELD-PadSH)")
+			(net "DGND")
 			(pinfunction "SHIELD_SH")
 			(pintype "passive")
@@
 			(layers "*.Cu" "*.Mask")
 			(remove_unused_layers no)
-			(net "unconnected-(J1-SHIELD-PadSH)")
+			(net "DGND")
 			(pinfunction "SHIELD_SH")
 			(pintype "passive")
@@
 			(layers "*.Cu" "*.Mask")
 			(remove_unused_layers no)
-			(net "unconnected-(J1-SHIELD-PadSH)")
+			(net "DGND")
 			(pinfunction "SHIELD_SH")
 			(pintype "passive")

Commit message: feat(v1 hardware): review fixes
Parts:
- D1, D10, D11, D12, D13, D14, D15, D16, D17, D18, D19, D2, D20, D21, D22, D23, D24, D25, D26, D27, D28, D29, D3, D30, D31, D32, D33, D34, D35, D36, D37, D38, D39, D4, D40, D41, D42, D43, D44, D45, D46, D47, D48, D49, D5, D50, D51, D52, D53, D54, D55, D56, D57, D58, D59, D6, D60, D61, D62, D63, D64, D65, D66, D67, D68, D69, D7, D70, D71, D72, D73, D74, D75, D76, D77, D78, D79, D8, D80, D81, D82, D9: value D -> BAS16TS
- JP2, JP3, JP4, JP5, JP6: moved to B.Cu
- R41, R45: value 13kΩ -> 22kΩ
- moved J3 170.9 mm to (238.8, 78.5)
- moved SW8 167.9 mm to (250.4, 73.1), turned to 45 degrees
- moved JP2 5.89 mm to (218.3, 250.4)
- moved JP3 5.89 mm to (222.9, 250.4)
- moved JP4 5.89 mm to (227.4, 250.4)
- moved JP5 0.70 mm to (213.3, 27.2)
- moved JP6 0.70 mm to (217.8, 27.2)
Connections:
- IC1 pad 12: unconnected-(IC1-PGND_2-Pad12) -> DGND
- IC1 pad 13: unconnected-(IC1-VOUT_2-Pad13) -> +5V
- IC1 pad 14: unconnected-(IC1-VIN_2-Pad14) -> V_IN_TPS
- IC1 pad 15: unconnected-(IC1-FB_2-Pad15) -> /Power Train/FB
